File: puissance.kicad_pcb (KiCad board)
At the start: 4 copper layers, 73.9 x 43 mm, 37 parts, among them J5 Screw_Terminal_01x10, J8 MEC1-110-02-F-D-A, J9 Screw_Terminal_01x04, K5 G6DN-1A-L DC24, K6 G6DN-1A-L DC24, U11 SIP-4_1779205311, U12 PDRV81545PWPR, U13 ISO7720D, U14 TLV75709PDBV, U8 ISO1212

Commit message: update
Parts:
- J8: moved to B.Cu
- moved L1 23.6 mm to (147.4, 55.9)
- moved C19 23.6 mm to (122.5, 75.4)
- moved RV4 23.6 mm to (118.0, 85.4)
- moved C21 23.6 mm to (103.7, 73.9)
- moved C15 23.6 mm to (150.6, 54.4)
- moved C17 23.6 mm to (151.0, 60.1)
- moved C18 23.6 mm to (155.0, 57.2)
- moved C22 23.6 mm to (103.7, 69.3)
- moved D8 23.6 mm to (114.9, 75.4)
- moved J5 23.6 mm to (106.0, 52.5)
- moved J9 23.6 mm to (106.0, 82.9)
- moved K5 23.6 mm to (132.0, 83.8)
- moved K6 23.6 mm to (132.0, 89.6)
- moved OC2 23.6 mm to (150.0, 86.7)
- moved R12 23.6 mm to (117.2, 62.7)
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Connections:
- J8 pad 07: unconnected-(J8-Pad07) -> /Relay1_MCU
- J8 pad 09: unconnected-(J8-Pad09) -> /Relay2_MCU
- J8 pad 11: unconnected-(J8-Pad11) -> /Output1_MCU
- J8 pad 15: unconnected-(J8-Pad15) -> /Output2_MCU
- J8 pad 17: unconnected-(J8-Pad17) -> /Input1_MCU
- J8 pad 19: unconnected-(J8-Pad19) -> /Input2_MCU
Routing:
- net +3V3: track 0.00 -> 47.7 mm
- net /Output2_MCU: track 0.00 -> 36.0 mm, vias 0 -> 1
- net GND1: track 2.09 -> 15.5 mm, vias 0 -> 2
- added copper zone on In1.Cu, net GND1
- removed copper zone on In1.Cu, net +3V3
- removed copper zone on In2.Cu, net GND1
Other:
- board size 73.9 x 43 mm -> 65 x 43 mm

Commit message: suite et nouvel écran
Parts:
- removed J9: Screw_Terminal_01x04, TerminalBlock_Phoenix:TerminalBlock_Phoenix_MPT-0,5-4-2.54_1x04_P2.54mm_Horizontal
- added C1: 47µ 50V, PCM_Capacitor_SMD_AKL:CP_Elec_6.3x7.7, F.Cu at (116.5, 62.6)
- added C23: 1µ, Capacitor_SMD:C_0603_1608Metric_Pad1.08x0.95mm_HandSolder, F.Cu at (111.3, 65.3)
- added C24: 0.1µ, Capacitor_SMD:C_0603_1608Metric_Pad1.08x0.95mm_HandSolder, F.Cu at (145.8, 63.9)
- added F1: 100mA, Fuse:Fuse_1812_4532Metric, F.Cu at (122.6, 53.5)
- added J2: Screw_Terminal_01x04, TerminalBlock_Phoenix:TerminalBlock_Phoenix_PT-1,5-4-3.5-H_1x04_P3.50mm_Horizontal, F.Cu at (107.4, 80.2)
- added R17: optional, Resistor_SMD:R_0805_2012Metric_Pad1.20x1.40mm_HandSolder, F.Cu at (132.4, 63.8)
- added R18: optional, Resistor_SMD:R_0805_2012Metric_Pad1.20x1.40mm_HandSolder, F.Cu at (132.4, 59.6)
- C13, C14: value 0.1µ -> 10n; footprint Capacitor_SMD:C_0603_1608Metric_Pad1.08x0.95mm_HandSolder -> Capacitor_SMD:C_0603_1608Metric
- R12, R15: value 562 -> 560; footprint Resistor_SMD:R_0603_1608Metric_Pad0.98x0.95mm_HandSolder -> Resistor_SMD:R_0603_1608Metric
- R13, R14: value 2k5 -> 2k4; footprint Resistor_SMD:R_0603_1608Metric_Pad0.98x0.95mm_HandSolder -> Resistor_SMD:R_0805_2012Metric_Pad1.20x1.40mm_HandSolder
- U13: value ISO7720D -> ISO6420FDR
- moved TP1 24.6 mm to (149.4, 65.4)
- moved TP2 24.6 mm to (149.3, 68.6)
- moved C14 20.5 mm to (135.0, 60.0), turned to 90 degrees
- moved C13 20.4 mm to (135.0, 64.2), turned to 90 degrees
- moved R15 19.5 mm to (136.6, 60.0), turned to -90 degrees
- moved R12 19.4 mm to (136.6, 64.2), turned to -90 degrees
- moved R14 16.3 mm to (128.0, 60.5)
- moved R13 16.2 mm to (128.0, 64.7)
- moved U8 7.63 mm to (141.1, 61.8)
- moved U13 3.28 mm to (136.2, 72.1)
- moved D8 1.72 mm to (113.2, 75.6)
- moved R16 1.35 mm to (123.2, 66.7), turned to 180 degrees
- moved RV3 1.08 mm to (118.9, 89.9)
- moved RV4 1.03 mm to (118.9, 84.9)
- moved D3 1.00 mm to (114.6, 53.5)
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Connections:
- net /Input1 renamed /Entrée/Input1
- net /Input2 renamed /Entrée/Input2
- net /Output1 renamed /Sorties/Output2
- net /Output2 renamed /Sorties/Output1
- net Net-(J9-Pin_1) renamed /Sorties/Relais2_COM
- net Net-(J9-Pin_2) renamed /Sorties/Relais2_NO
- net Net-(J9-Pin_3) renamed /Sorties/Relais1_COM
- net Net-(J9-Pin_4) renamed /Sorties/Relais1_NO
- C13 pad 1: Net-(U8-IN1) -> Net-(U8-SENSE1)
- C14 pad 1: Net-(U8-IN2) -> Net-(U8-SENSE2)
- D3 pad 1: +24V -> Net-(D3-K)
- D8 pad 2: /Voutput -> GND2
- J5 pad 10: /Voutput -> unconnected-(J5-Pin_10-Pad10)
- J8 pad 07: /Relay1_MCU -> /Output_6
- J8 pad 08: unconnected-(J8-Pad08) -> /Output_6
- J8 pad 09: /Relay2_MCU -> /Output_5
- J8 pad 10: unconnected-(J8-Pad10) -> /Output_5
- J8 pad 11: /Output1_MCU -> /Output_4
- J8 pad 12: unconnected-(J8-Pad12) -> /Output_4
- J8 pad 15: /Output2_MCU -> /Output_3
- J8 pad 16: unconnected-(J8-Pad16) -> /Output_3
- J8 pad 17: /Input1_MCU -> /Output_2
- J8 pad 18: unconnected-(J8-Pad18) -> /Output_2
- J8 pad 19: /Input2_MCU -> /Output_1
- J8 pad 20: unconnected-(J8-Pad20) -> /Output_1
- R12 pad 1: Net-(U8-SENSE1) -> Net-(U8-IN1)
- R12 pad 2: Net-(U8-IN1) -> Net-(U8-SENSE1)
- R13 pad 2: Net-(U8-IN1) -> Net-(U8-SENSE1)
- R14 pad 2: Net-(U8-IN2) -> Net-(U8-SENSE2)
- R15 pad 1: Net-(U8-SENSE2) -> Net-(U8-IN2)
- R15 pad 2: Net-(U8-IN2) -> Net-(U8-SENSE2)
- R23 pad 1: /Relay1_MCU -> /Output_1
- R24 pad 1: /Relay2_MCU -> /Output_2
- U13 pad 2: /Output1_MCU -> /Sorties/Output1_MCU
- U13 pad 3: /Output2_MCU -> /Sorties/Output2_MCU
Routing:
- net +3V3: track 47.7 -> 0.00 mm
- net /Output2_MCU: track 36.0 -> 0.00 mm, vias 1 -> 0
- net /Output_3: track 0.00 -> 28.6 mm
- net Net-(D8-K): track 0.00 -> 18.0 mm
- net GND2: track 0.00 -> 13.0 mm, vias 0 -> 13
- net +24V: track 6.73 -> 16.4 mm, vias 0 -> 6
- net /Sorties/Output2: track 0.00 -> 7.13 mm
- net Net-(D3-A): track 0.00 -> 7.01 mm
- net /Sorties/Output1: track 0.00 -> 6.84 mm
- net Net-(U12A-ILIM): track 0.00 -> 4.28 mm
- net Net-(D3-K): track 0.00 -> 3.86 mm
- net /Sorties/Relais1_COM: track 26.9 -> 25.5 mm
- net /Sorties/Relais1_NO: track 18.0 -> 17.1 mm
- net /Sorties/Relais2_NO: track 18.0 -> 17.3 mm
- net Net-(U8-SUB2): track 0.00 -> 0.70 mm
- added copper zone on F.Cu, net +24V
- added copper zone on F.Cu, net GND2

Commit message: corrections
Parts:
- added C10: 0.1µ, Capacitor_SMD:C_0603_1608Metric_Pad1.08x0.95mm_HandSolder, F.Cu at (139.3, 72.6)
- added C9: 0.1µ, Capacitor_SMD:C_0603_1608Metric_Pad1.08x0.95mm_HandSolder, F.Cu at (149.6, 71.7)
- added D5: SMAJ33CA, PCM_Diode_SMD_AKL:D_SMA_TVS, F.Cu at (132.2, 53.5)
- added J4: Screw_Terminal_01x04, TerminalBlock_Phoenix:TerminalBlock_Phoenix_MKDS-3-4-5.08_1x04_P5.08mm_Horizontal, F.Cu at (3.06, 6.42)
- added Q2: 2N7002, PCM_Package_TO_SOT_SMD_AKL:SOT-23, F.Cu at (144.5, 89.3)
- added Q3: 2N7002, PCM_Package_TO_SOT_SMD_AKL:SOT-23, F.Cu at (144.5, 83.5)
- added R10: 47k, Resistor_SMD:R_0603_1608Metric_Pad0.98x0.95mm_HandSolder, F.Cu at (147.3, 89.4)
- added R11: 470, Resistor_SMD:R_0603_1608Metric_Pad0.98x0.95mm_HandSolder, F.Cu at (148.9, 89.4)
- added R12: 47k, Resistor_SMD:R_0603_1608Metric_Pad0.98x0.95mm_HandSolder, F.Cu at (147.3, 83.6)
- added R13: 470, Resistor_SMD:R_0603_1608Metric_Pad0.98x0.95mm_HandSolder, F.Cu at (148.9, 83.6)
- U3: renamed from U12; value PDRV81545PWPR -> DRV81545PWPR
- U5: renamed from U14; value TLV75709PDBV -> TLV709
- moved C12 8.88 mm to (135.7, 73.3)
- moved TP1 8.71 mm to (142.7, 59.8)
- moved U4 8.13 mm to (144.0, 69.8)
- moved TP2 7.97 mm to (142.7, 64.2)
- moved U5 7.84 mm to (132.6, 73.4), turned to 0 degrees
- moved C11 7.23 mm to (129.4, 73.3)
- moved OC1 4.20 mm to (154.2, 86.2)
- moved R8 4.20 mm to (160.1, 85.6)
- moved R9 4.20 mm to (160.2, 88.1)
- moved C13 3.63 mm to (158.6, 57.8)
- moved C1 3.20 mm to (147.3, 55.3)
- moved C2 3.20 mm to (153.7, 55.3)
- moved L1 3.20 mm to (150.5, 56.8)
- moved C4 3.20 mm to (154.1, 61.0)
- moved U1 3.20 mm to (156.1, 54.2)
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- renumbered C16 to C1, C19 to C11, C20 to C12, C18 to C13, C22 to C14, C21 to C15, C15 to C2, C14 to C3, C17 to C4, C1 to C5, C13 to C6, C24 to C7, C23 to C8, D3 to D1, D8 to D2, D7 to D3, D6 to D4, J5 to J1, J8 to J3, K5 to K1, K6 to K2, OC2 to OC1, R18 to R1, R15 to R2, R14 to R3, R17 to R4, R12 to R5, R13 to R6, R16 to R7, R24 to R8, R23 to R9, RV4 to RV1, RV3 to RV2, U11 to U1, U8 to U2, U13 to U4
Connections:
- C12 pad 1: Net-(U13-VCC2) -> +5VP
- C13 pad 2: Net-(U11-+VIN) -> GND2
- C2 pad 1: Net-(U11-+VIN) -> Net-(U1-+VIN)
- D3 pad 2: Net-(D7-A) -> Net-(D3-A)
- D4 pad 2: Net-(D6-A) -> Net-(D4-A)
- J1 pad 10: unconnected-(J5-Pin_10-Pad10) -> GND2
- J1 pad 7: GND2 -> /Sorties/Output1
- J1 pad 8: /Sorties/Output1 -> GND2
- K1 pad A1: Net-(D7-A) -> Net-(D3-A)
- K2 pad A1: Net-(D6-A) -> Net-(D4-A)
- L1 pad 2: Net-(U11-+VIN) -> Net-(U1-+VIN)
- OC1 pad 5: GND2 -> Net-(OC1-Pad5)
- OC1 pad 6: Net-(D7-A) -> +5VP
- OC1 pad 7: GND2 -> Net-(OC1-Pad7)
- OC1 pad 8: Net-(D6-A) -> +5VP
- U1 pad 2: Net-(U11-+VIN) -> Net-(U1-+VIN)
- U2 pad 4: /Input1_MCU -> /Output_5
- U2 pad 5: /Input2_MCU -> /Output_6
- U4 pad 2: /Sorties/Output1_MCU -> /Output_3
- U4 pad 3: /Sorties/Output2_MCU -> /Output_4
- U4 pad 8: Net-(U13-VCC2) -> +5VP
- U5 pad 5: Net-(U13-VCC2) -> +5VP
Routing:
- net GND2: track 13.0 -> 64.8 mm, vias 13 -> 42
- net +3V3: track 0.00 -> 39.6 mm, vias 0 -> 3
- net +5VP: track 0.00 -> 38.9 mm
- net /Entrée/Input2: track 0.00 -> 30.3 mm
- net /Output_5: track 0.00 -> 30.1 mm, vias 0 -> 2
- net /Output_6: track 0.00 -> 29.9 mm, vias 0 -> 2
- net /Output_4: track 0.00 -> 27.8 mm, vias 0 -> 2
- net /Entrée/Input1: track 0.00 -> 25.6 mm
- net Net-(U3A-IN1): track 0.00 -> 24.6 mm
- net /Output_1: track 0.00 -> 24.5 mm, vias 0 -> 1
- net Net-(U3A-IN3): track 0.00 -> 24.4 mm
- net /Output_2: track 0.00 -> 23.2 mm, vias 0 -> 1
- net Net-(U2-SENSE1): track 0.00 -> 10.1 mm
- net Net-(D6-A): track 10.0 -> 0.00 mm
- net Net-(U2-SENSE2): track 0.00 -> 9.61 mm
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- added copper zone on B.Cu, net +5VD
- added copper zone on B.Cu, net GND1
- added copper zone on F.Cu, net GND1
- added copper zone on In2.Cu, net GND1
- added copper zone on B.Cu, net GND2
Other:
- outline, holes or cut-outs redrawn

Commit message: daily
Parts:
- removed J4: Screw_Terminal_01x04, TerminalBlock_Phoenix:TerminalBlock_Phoenix_MKDS-3-4-5.08_1x04_P5.08mm_Horizontal
- C12: value 0.47µ -> 1µ
- F1: footprint Fuse:Fuse_1812_4532Metric -> Fuse:Fuse_1210_3225Metric
- U5: value TLV709 -> TLV709A50DBVR
- moved D2 4.20 mm to (128.0, 53.3)
- moved F1 3.13 mm to (119.5, 53.1)
- moved D1 1.26 mm to (113.4, 53.1)
- moved TP1 1.10 mm to (143.8, 59.8)
- moved TP2 1.10 mm to (143.8, 64.2)
- moved C13 0.41 mm to (159.0, 58.0)
- renumbered D5 to D2, D2 to D3, D3 to D4, D4 to D5, Q3 to Q1, R8 to R10, R9 to R11, R10 to R12, R11 to R13, R12 to R8, R13 to R9
Connections:
- J3 pad 08: /Output_6 -> unconnected-(J3-Pad08)
- J3 pad 10: /Output_5 -> unconnected-(J3-Pad10)
- J3 pad 12: /Output_4 -> unconnected-(J3-Pad12)
- J3 pad 16: /Output_3 -> unconnected-(J3-Pad16)
- J3 pad 17: /Output_2 -> unconnected-(J3-Pad17)
- J3 pad 19: /Output_1 -> unconnected-(J3-Pad19)
Routing:
- net GND2: track 64.8 -> 60.7 mm
- net /Output_4: track 27.8 -> 24.9 mm, vias 2 -> 1
- net /Output_3: track 28.1 -> 25.2 mm, vias 2 -> 1
- net /Output_5: track 30.1 -> 27.2 mm, vias 2 -> 1
- net /Output_2: track 23.2 -> 20.2 mm, vias 1 -> 0
- net /Output_1: track 24.5 -> 21.6 mm, vias 1 -> 0
- net /Output_6: track 29.9 -> 27.0 mm, vias 2 -> 1
- net Net-(D1-A): track 7.01 -> 5.65 mm
- net Net-(D1-K): track 3.86 -> 2.70 mm
Other:
- board text added: "JLCJLCJLC"
- board text added: "OPC V0.2 - GaOu 2026"

Commit message: daily
Parts:
- removed J1: Screw_Terminal_01x10, TerminalBlock_Phoenix:TerminalBlock_Phoenix_MPT-0,5-10-2.54_1x10_P2.54mm_Horizontal
- removed J2: Screw_Terminal_01x04, TerminalBlock_Phoenix:TerminalBlock_Phoenix_PT-1,5-4-3.5-H_1x04_P3.50mm_Horizontal
- added J4: 1705566, OPC:1705566, F.Cu at (108.5, 78.8)
- added J5: 1725672, OPC:1725672, F.Cu at (103.6, 64.8)
- added J6: 1725672, OPC:1725672, F.Cu at (103.6, 52.0)
- added JP1: SolderJumper_2_Open, Jumper:SolderJumper-2_P1.3mm_Open_RoundedPad1.0x1.5mm, F.Cu at (117.8, 73.5)
- C10, C7, C9: value 0.1µ -> 0.1µ 10V
- C11: value 0.1µ -> 0.1µ 50V
- C12, C8: value 1µ -> 1µ 50V; footprint Capacitor_SMD:C_0603_1608Metric_Pad1.08x0.95mm_HandSolder -> Capacitor_SMD:C_0805_2012Metric_Pad1.18x1.45mm_HandSolder
- C14, C15: value 10n -> 10n 100V; footprint Capacitor_SMD:C_0805_2012Metric_Pad1.18x1.45mm_HandSolder -> Capacitor_SMD:C_0603_1608Metric_Pad1.08x0.95mm_HandSolder
- C3, C6: value 10n -> 10n 100V
- D1, D4, D5: value US1M -> FR1G
- D3: moved to B.Cu
- moved D3 4.80 mm to (108.8, 73.4)
- moved C14 3.77 mm to (101.7, 66.1)
- moved C15 3.44 mm to (101.7, 71.1)
- moved C8 3.24 mm to (108.8, 63.4), turned to 90 degrees
- moved C5 2.28 mm to (114.5, 61.5)
- moved U3 2.20 mm to (113.0, 68.7)
- moved R7 2.20 mm to (120.9, 64.8)
- moved U5 1.64 mm to (131.6, 72.1)
- moved C11 1.64 mm to (128.4, 72.0)
- moved C12 1.52 mm to (134.7, 72.2)
- moved F1 0.20 mm to (119.5, 53.3)
- moved C13 0.06 mm to (159.0, 58.0)
Routing:
- net GND2: track 60.7 -> 43.7 mm, vias 42 -> 43
- net /Sorties/Relais2_NO: track 16.9 -> 22.0 mm
- net /Sorties/Relais2_COM: track 26.0 -> 30.9 mm
- net /Sorties/Relais1_COM: track 25.5 -> 30.2 mm
- net /Sorties/Relais1_NO: track 17.0 -> 21.1 mm
- net /Entrée/Input1: track 25.6 -> 28.5 mm
- net Net-(D1-A): track 5.65 -> 8.26 mm
- net +5VP: track 38.9 -> 41.4 mm
- net Net-(U3A-IN1): track 24.6 -> 27.0 mm
- net Net-(U3A-IN3): track 24.4 -> 26.7 mm
- net Net-(D3-K): track 16.3 -> 15.1 mm, vias 0 -> 3
- net /Sorties/Output1: track 9.25 -> 10.1 mm
- net +24V: track 21.9 -> 21.3 mm, vias 16 -> 19
- net /Sorties/Output2: track 9.45 -> 8.94 mm
- added copper zone on B.Cu, net Net-(D3-K)
- added copper zone on F.Cu, net Net-(D3-K)
Other:
- outline, holes or cut-outs redrawn
- board text removed: "+"
- board text removed: "-"
- board text removed: "1"
- board text removed: "2"
- board text removed: "In1"
- board text removed: "In2"
- board text removed: "O1"
- board text removed: "O2"
- board text removed: "V+"
- board text removed: "V-"
- board text removed: "Vin"

Commit message: avant prod
Parts:
- R3, R6: value 2k4 -> 1000; footprint Resistor_SMD:R_0805_2012Metric_Pad1.20x1.40mm_HandSolder -> Resistor_SMD:R_1206_3216Metric
- U1: value SIP-4_1779205311 -> 1779205311; footprint PCM_MagIC_THT_Wurth:U_Wurth_WPME-FISM-SIP-4_1779405311 -> PCM_MagIC_THT_Wurth:U_Wurth_WPME-FISM-SIP-4_1779205311
- moved R3 1.11 mm to (129.8, 60.9)
- moved R6 1.11 mm to (129.8, 65.1)
- moved C5 0.45 mm to (115.0, 61.5)
- moved D4 0.20 mm to (139.1, 81.6)
- moved K1 0.20 mm to (132.0, 83.1)
- moved RV1 0.20 mm to (118.9, 83.3)
Connections:
- C14 pad 1: /Sorties/Output1 -> /Sorties/Output2
- C15 pad 1: /Sorties/Output2 -> /Sorties/Output1
- J5 pad 1: /Sorties/Output1 -> /Sorties/Output2
- J5 pad 3: /Sorties/Output2 -> /Sorties/Output1
- J6 pad 3: /Entrée/Input1 -> /Entrée/Input2
- J6 pad 4: /Entrée/Input2 -> /Entrée/Input1
- R3 pad 1: /Entrée/Input1 -> /Entrée/Input2
- R6 pad 1: /Entrée/Input2 -> /Entrée/Input1
- U3 pad 14: /Sorties/Output1 -> /Sorties/Output2
- U3 pad 15: /Sorties/Output1 -> /Sorties/Output2
- U3 pad 16: /Sorties/Output2 -> /Sorties/Output1
- U3 pad 17: /Sorties/Output2 -> /Sorties/Output1
Routing:
- net /Entrée/Input2: track 30.7 -> 28.0 mm
- net /Entrée/Input1: track 28.5 -> 30.0 mm
- net /Sorties/Output1: track 10.1 -> 8.93 mm
- net /Sorties/Output2: track 8.94 -> 10.1 mm
- net Net-(U2-SENSE1): track 10.1 -> 10.7 mm
- net Net-(U2-SENSE2): track 9.61 -> 10.2 mm
- net +24V: track 21.3 -> 20.7 mm
