File: OPC V3.kicad_sch (KiCad schematic)
At the start: 0 parts

Commit message: MAJ post prod
Other:
- note added: "Consommation : 20mA @ 24V ~= 0.5W"
- note added: "Erreurs V0.2 : - RREF1k65 & RREF16k5 inversés dans le schémas général Sensor Board. -> Fix 0.2 : inverser le gpio correspondant dans le code (pinout.h) -> Fix 0.3 : Changer le cablage sur la page 1 de Sensor board - Les connecteurs entrées ne sont pas assez près du bord, quand on insère les fiches, elles touchent le pcb -> Fix 0.2 : En jouant avec ça rentre quand même. -> Fix 0.3 : Déplacer les c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"
