File: connecteur.kicad_sch (KiCad schematic)
At the start: 1 part, among them J7 MEC1-110-02-F-D-A

Commit message: suite et nouvel écran
Parts:
- renumbered J7 to J3
Connections:
- net OUTPUT_4: now also J3.12; no longer J3.08
- net OUTPUT_5: now also J3.10; no longer J3.12
- net OUTPUT_6: now also J3.08; no longer J3.10
Changed lines of the file:
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@@
 		)
 	)
-	(hierarchical_label "OUTPUT_6"
+	(hierarchical_label "OUTPUT_5"
 		(shape input)
 		(at 166.37 91.44 0)
@@
 		)
 	)
-	(hierarchical_label "OUTPUT_5"
+	(hierarchical_label "OUTPUT_4"
 		(shape input)
 		(at 166.37 93.98 0)
@@
 		)
 	)
-	(hierarchical_label "OUTPUT_4"
+	(hierarchical_label "OUTPUT_6"
 		(shape input)
 		(at 166.37 88.9 0)
@@
 		(dnp no)
 		(fields_autoplaced yes)
-		(property "Reference" "J7"
+		(property "Reference" "J3"
 			(at 148.59 73.66 0)
 			(show_name no)
@@
 			(project "OPC V2"
 				(path "/594181e6-a34f-458c-9685-d994528736df/cb01c09e-2b15-40e2-9aed-1b8210bf4dac"
-					(reference "J7")
+					(reference "J3")
 					(unit 1)
 				)

Commit message: corrections
Parts:
- J3: now left out of the parts list
Changed lines of the file:
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@@
 		(body_style 1)
 		(exclude_from_sim no)
-		(in_bom yes)
+		(in_bom no)
 		(on_board yes)
-		(in_pos_files yes)
+		(in_pos_files no)
 		(dnp no)
 		(fields_autoplaced yes)

Commit message: daily
Other:
- title: (none) -> Connecteur pcb
Changed lines of the file:
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@@
 	(generator_version "10.0")
 	(paper "A4")
+	(title_block
+		(title "Connecteur pcb")
+	)
 	(rectangle
 		(start 99.06 69.85)
@@
 			)
 		)
+		(property "px_x10" ""
+			(at 148.59 93.98 0)
+			(hide yes)
+			(show_name no)
+			(do_not_autoplace no)
+			(effects
+				(font
+					(size 1.27 1.27)
+				)
+			)
+		)

Commit message: daily
Parts:
- J3: now in the parts list
Changed lines of the file:
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@@
 		(body_style 1)
 		(exclude_from_sim no)
-		(in_bom no)
+		(in_bom yes)
 		(on_board yes)
-		(in_pos_files no)
+		(in_pos_files yes)
 		(dnp no)
 		(fields_autoplaced yes)
