File: ecran_FPC.kicad_sch (KiCad schematic)
At the start: 17 parts, among them J6 MEC1-110-02-F-D-A, J8 MEC1-110-02-F-D-A, SW1 PEC11L-4220K-S0015

Commit message: suite et nouvel écran
Parts:
- removed R11: 47, Resistor_SMD:R_0603_1608Metric_Pad0.98x0.95mm_HandSolder, symbol Device:R
- removed U8: (no value), OPC:WAVESHARE-1.14-LCD-2, symbol OPC:WAVESHARE-1.14-LCD
- added C16: 4µ7 50V, Capacitor_SMD:C_1206_3216Metric, symbol Device:C_Small
- added J1: 1-2328724-5, 123287245, symbol OPC:1-2328724-5
- added JP2: SolderJumper_2_Open, Jumper:SolderJumper-2_P1.3mm_Open_RoundedPad1.0x1.5mm, symbol Jumper:SolderJumper_2_Open
- added R1: 10, PCM_Resistor_SMD_AKL:R_1206_3216Metric_Pad1.30x1.75mm, symbol Device:R
- added R15: 47, Resistor_SMD:R_0603_1608Metric_Pad0.98x0.95mm_HandSolder, symbol Device:R
- added R19, R20: 6k8, Resistor_SMD:R_0603_1608Metric_Pad0.98x0.95mm_HandSolder, symbol Device:R
- C13, C14, C15: value 0.1µ -> 10n; LCSC Part # C14663 -> C57112
Connections:
- net +3.3V: now also C16.1, J1.3, J1.4, JP2.1 (A), R1.1
- net LCD_CLK: now also R15.2; no longer R12.1
- net LCD_DIN: now also R12.2
- net ROTENC_+: now also R19.1; no longer C15.2, R18.2, SW1.A
- net ROTENC_-: now also R20.2; no longer C14.2, R17.2, SW1.B
- net at R13.2: now also J1.8
- net at R14.2: now also J1.10
- net GND1 renamed GND
- net GND: now also C16.2, J1.13, J1.14, J1.15, J1.2, J1.5, J1.6
- new net: C14.2, R17.2, R20.1, SW1.B
- new net: J1.1, R1.2
- new net: C15.2, R18.2, R19.2, SW1.A
- new net: J1.9, R15.1
- new net: J1.7, JP2.2 (B)
- new net: J1.11, R12.1
Other:
- moved on the sheet: C12, J6, J8, R12, R13, R14

Commit message: corrections
Parts:
- removed JP2: SolderJumper_2_Open, Jumper:SolderJumper-2_P1.3mm_Open_RoundedPad1.0x1.5mm, symbol Jumper:SolderJumper_2_Open
- added C1: 1µ, Capacitor_SMD:C_0603_1608Metric_Pad1.08x0.95mm_HandSolder, symbol Device:C_Small
- added R1: 10k, Resistor_SMD:R_0603_1608Metric_Pad0.98x0.95mm_HandSolder, symbol Device:R
- added TP1: TestPoint, TestPoint:TestPoint_Pad_1.5x1.5mm, symbol Connector:TestPoint
- C4: renamed from C15; value 10n -> 0.1u; LCSC Part # C57112 -> C14663
- C5: renamed from C14; value 10n -> 0.1u; LCSC Part # C57112 -> C14663
- J3: renamed from J1; footprint 123287245 -> OPC:123287245
- SW1: footprint Rotary_Encoder:RotaryEncoder_Alps_EC11E-Switch_Vertical_H20mm_MountingHoles -> OPC:PEC11L4220KS0015
- renumbered C16 to C2, C12 to C3, C13 to C6, J6 to J1, J8 to J2, R17 to R10, R18 to R11, R1 to R2, R19 to R3, R15 to R4, R12 to R5, R14 to R6, R13 to R7, R20 to R8, R16 to R9
Connections:
- net +3.3V: now also R1.2
- net GND: now also C1.2
- net OUTPUT_4: now also J1.12, J2.11, J2.12; no longer J1.08, J2.07, J2.08
- net OUTPUT_5: now also J1.10, J2.09, J2.10; no longer J1.12, J2.11, J2.12
- net OUTPUT_6: now also J1.08, J2.07, J2.08; no longer J1.10, J2.09, J2.10
- net at J3.7: now also C1.1, R1.1, TP1.1
Other:
- note added: "Connecteur vers carte mesure"
- note added: "Connecteur vers carte puissance"
- note added: "Ecran LCD 1.54" IPS (MIKROE-6588)"
- note added: "Fixation pcb"
- note added: "Rotary encoder + filtering"
- note removed: "Rotary encoder"
- moved on the sheet: C2, C3, C4, C5, C6, H1, H2, J1, J2, R10, R11, R3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

Commit message: daily
Parts:
- added U1: IPS 240*240 display, symbol Display_Graphic:ER_OLEDM0.91_1x-I2C
- C1: MF (none) -> Murata; MPN (none) -> GRM033R60G105MEA2D; px_1 (none) -> 0,086; px_10 (none) -> 0,034
- C2: value 4µ7 50V -> 4µ7; footprint Capacitor_SMD:C_1206_3216Metric -> Capacitor_SMD:C_0805_2012Metric_Pad1.18x1.45mm_HandSolder; MPN (none) -> GRM21BR71A475KE51K; px_1 (none) -> 0,103; px_10 (none) -> 0,039
- C3: MF (none) -> Würth Elektronik; MPN (none) -> 885012206020; px_1 (none) -> 0,095; px_10 (none) -> 0.031
- C4, C5: value 0.1u -> 0.1µ; MF (none) -> Würth Elektronik; MPN (none) -> 885012206020; px_1 (none) -> 0,095; px_10 (none) -> 0.031
- C6: value 10n -> 0.1µ; LCSC Part # C57112 -> C14663; MPN (none) -> 885012206020; px_1 (none) -> 0,095; px_10 (none) -> 0.031
- J1, J2: MPN (none) -> MEC1-110-02-F-D-A; px_1 (none) -> 3,47
- J3: MF (none) -> TE Connectivity; MPN (none) -> 1-2328724-5; px_1 (none) -> 0,249; px_10 (none) -> 0.215
- R1: MF (none) -> Panasonic; MPN (none) -> ERJ-3EKF1002V; px_1 (none) -> 0,086; px_10 (none) -> 0.021
- R10, R11, R3, R8, R9: MF (none) -> Panasonic; MPN (none) -> ERJ-3EKF6801V; px_1 (none) -> 0,086; px_10 (none) -> 0.021
- R2: MF (none) -> Panasonic; MPN (none) -> ERJ-U08J100V; px_1 (none) -> 0,146; px_10 (none) -> 0.048
- R4, R5, R6, R7: MF (none) -> Panasonic; MPN (none) -> ERJ-3GEYJ470V; px_1 (none) -> 0,086; px_10 (none) -> 0.02
- SW1: MF (none) -> Bourns; MPN (none) -> PEC11L-4220K-S0015; px_1 (none) -> 2.13; px_10 (none) -> 1.78
- TP1: now left out of the parts list

Commit message: daily
Parts:
- removed U1: IPS 240*240 display, symbol Display_Graphic:ER_OLEDM0.91_1x-I2C
- added U2: IPS_240x240, FPC 15 - 0.3mm, symbol OPC:IPS_240x240
- C1: value 1µ -> 1µ 50V; footprint Capacitor_SMD:C_0603_1608Metric_Pad1.08x0.95mm_HandSolder -> Capacitor_SMD:C_0805_2012Metric_Pad1.18x1.45mm_HandSolder; LCSC Part # C15849 -> C28323; MPN GRM033R60G105MEA2D -> GRM219R61H105MA73D; px_1 0,086 -> 0.129; px_10 0,034 -> 0.052
- C2: value 4µ7 -> 4µ7 10V
- C3, C4, C5: value 0.1µ -> 0.1µ 10V
- C6: value 0.1µ -> 0.1µ 10V; MF (none) -> Würth Elektronik
Other:
- note added: "Connecteur FPC pour écran (MIKROE-6588)"
- note removed: "Ecran LCD 1.54" IPS (MIKROE-6588)"
- moved on the sheet: C4, C5, C6, J2, R10, R11, R3, R6, R7, R8, R9, SW1

Commit message: avant prod
Parts:
- C2: LCSC Part # C29823 -> C1779
Changed lines of the file:
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@@
 			)
 		)
-		(property "LCSC Part #" "C29823"
+		(property "LCSC Part #" "C1779"
 			(at 38.1 43.18 0)
 			(hide yes)

Commit message: pre prod
Parts:
- SW1: value PEC11L-4220K-S0015 -> PEC11L-4220F-S0015; MPN PEC11L-4220K-S0015 -> PEC11L-4220F-S0015; px_1 2.13 -> 2.35; px_10 1.78 -> 2.02
Changed lines of the file:
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@@
 			)
 		)
-		(property "Value" "PEC11L-4220K-S0015"
+		(property "Value" "PEC11L-4220F-S0015"
 			(at 227.33 62.2299 90)
 			(hide yes)
@@
 			)
 		)
-		(property "MPN" "PEC11L-4220K-S0015 "
+		(property "MPN" "PEC11L-4220F-S0015 "
 			(at 233.68 60.96 90)
 			(hide yes)
@@
 			)
 		)
-		(property "px_1" "2.13"
+		(property "px_1" "2.35"
 			(at 233.68 60.96 90)
 			(hide yes)
@@
 			)
 		)
-		(property "px_10" "1.78"
+		(property "px_10" "2.02"
 			(at 233.68 60.96 90)
 			(hide yes)

Commit message: MAJ post prod
Other:
- title: (none) -> Carte mère / HMI
Changed lines of the file:
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@@
 	(generator_version "10.0")
 	(paper "A4")
+	(title_block
+		(title "Carte mère / HMI")
+		(date "2026-08-17")
+		(rev "0.2")
+	)
 	(rectangle
 		(start 187.96 99.06)
