File: entrees.kicad_sch (KiCad schematic)
At the start: 17 parts, among them J1 691382010004, J2 691382010004, J3 691382010004, U1 TS3A4751PWR, U2 TS3A4751PWR, U3 TS3A4751PWR, U4 TS3A4751PWR, U5 TS3A4751PWR

Commit message: update
Connections:
- net 16k5 renamed RREF_16k5
- net 3k3 renamed RREF_1k65
Other:
- note added: "R1 & R2 => Low ppm/K !"
- note removed: "[R1;R4] => Low ppm/K !"
Changed lines of the file:
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@@
 		)
 	)
-	(text "[R1;R4] => Low ppm/K !"
+	(text "R1 & R2 => Low ppm/K !"
 		(exclude_from_sim no)
 		(at 235.966 117.856 0)
@@
 		)
 	)
-	(hierarchical_label "16k5"
+	(hierarchical_label "RREF_16k5"
 		(shape input)
 		(at 193.04 139.7 0)
@@
 		)
 	)
-	(hierarchical_label "3k3"
+	(hierarchical_label "RREF_1k65"
 		(shape input)
 		(at 193.04 137.16 0)

Commit message: suite et nouvel écran
Parts:
- added R6: 3k3, Resistor_SMD:R_0603_1608Metric_Pad0.98x0.95mm_HandSolder, symbol Device:R
- R7: renamed from R1; value 1k65 -> 3k3
- renumbered C3 to C11, C1 to C2, C4 to C3, C5 to C7, C2 to C8, J3 to J4, R3 to R1, U4 to U1, U1 to U2, U5 to U4, U2 to U6, U3 to U9
Connections:
- net GND: now also R6.2
- net at R7.1, U4.2 (COM1): now also R6.1
Other:
- note added: "R2 & R6 & R7 => Low ppm/K !"
- note removed: "R1 & R2 => Low ppm/K !"
- moved on the sheet: R1, R2, R4, R7

Commit message: corrections
Changed lines of the file:
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@@
 	)
 	(hierarchical_label "AINP"
-		(shape passive)
+		(shape bidirectional)
 		(at 158.75 129.54 180)
 		(effects
@@
 	)
 	(hierarchical_label "AINP"
-		(shape passive)
+		(shape bidirectional)
 		(at 83.82 53.34 0)
 		(effects
@@
 	)
 	(hierarchical_label "AINP"
-		(shape passive)
+		(shape bidirectional)
 		(at 60.96 133.35 180)
 		(effects
@@
 	)
 	(hierarchical_label "AINP"
-		(shape passive)
+		(shape bidirectional)
 		(at 236.22 53.34 0)
 		(effects
@@
 	)
 	(hierarchical_label "AINP"
-		(shape passive)
+		(shape bidirectional)
 		(at 160.02 53.34 0)
 		(effects

Commit message: daily
Parts:
- C11, C2, C3, C7, C8: value 0.1µ -> 0.1µ 10V; MF (none) -> Würth Elektronik; MPN (none) -> 885012206020; px_x1 (none) -> 0,095; px_x10 (none) -> 0.031
- J1, J2, J4: MPN (none) -> 691382010004; px_x1 (none) -> 1.1+3.47; px_x10 (none) -> 0.98+3.07
- R1, R4: MF (none) -> Panasonic; MPN (none) -> ERJ-3EKF1004V; px_x1 (none) -> 0,086; px_x10 (none) -> 0,021
- R2: MF (none) -> Panasonic; MPN (none) -> ERA-3ARB1652V; px_x1 (none) -> 0.619; px_x10 (none) -> 0,446
- R6, R7: MF (none) -> Panasonic; MPN (none) -> ERA-3ARB332V; px_x1 (none) -> 0.344; px_x10 (none) -> 0,25
- U1, U2, U4, U6, U9: MPN (none) -> TS3A4751PWR; px_x1 (none) -> 1,49; px_x10 (none) -> 1.09
Other:
- note added: "10ppm/K en standard (5ppm/K ou moins sont bcp plus cher)"
- title: (none) -> Entrées

Commit message: daily
Parts:
- R3: renamed from R1; px_x10 0,021 -> 0.02
- R7: renamed from R4; px_x10 0,021 -> 0.02
- renumbered R6 to R10, R2 to R5, R7 to R9
Changed lines of the file:
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@@
 			)
 		)
-		(property "MPN" "TS3A4751PWR "
+		(property "px_x1" "1,49"
 			(at 142.24 60.96 0)
 			(hide yes)
@@
 			)
 		)
-		(property "px_x1" "1,49"
+		(property "px_x10" "1.09"
 			(at 142.24 60.96 0)
 			(hide yes)
@@
 			)
 		)
-		(property "px_x10" "1.09"
+		(property "MPN" "TS3A4751PWR "
 			(at 142.24 60.96 0)
 			(hide yes)
@@
 		(dnp no)
 		(fields_autoplaced yes)
-		(property "Reference" "R6"
+		(property "Reference" "R10"
 			(at 207.01 109.22 90)
 			(show_name no)
@@
 			)
 		)
-		(property "MF" "Panasonic"
+		(property "px_x1" "0.344"
 			(at 207.01 115.57 90)
 			(hide yes)
@@
 			)
 		)
-		(property "MPN" "ERA-3ARB332V"
+		(property "px_x10" "0,25"
 			(at 207.01 115.57 90)
 			(hide yes)
@@
 			)
 		)
-		(property "px_x1" "0.344"
+		(property "MF" "Panasonic"
 			(at 207.01 115.57 90)
 			(hide yes)
@@
 			)
 		)
-		(property "px_x10" "0,25"
+		(property "MPN" "ERA-3ARB332V"
 			(at 207.01 115.57 90)
 			(hide yes)
@@
 			(project "OPC V2"
 				(path "/594181e6-a34f-458c-9685-d994528736df/e6add8e5-d5b5-453a-af59-4f27d08ef450"
-					(reference "R6")
+					(reference "R10")
 					(unit 1)
 				)
@@
 		(dnp no)
 		(fields_autoplaced yes)
-		(property "Reference" "R4"
+		(property "Reference" "R7"
 			(at 233.68 125.73 90)
 			(show_name no)
@@
 			)
 		)
-		(property "MF" "Panasonic"
+		(property "px_x1" "0,086"
 			(at 233.68 132.08 90)
 			(hide yes)
@@
 			)
 		)
-		(property "MPN" "ERJ-3EKF1004V"
+		(property "px_x10" "0.02"
 			(at 233.68 132.08 90)
 			(hide yes)
@@
 			)
 		)
-		(property "px_x1" "0,086"
+		(property "MF" "Panasonic"
 			(at 233.68 132.08 90)
 			(hide yes)
@@
 			)
 		)
-		(property "px_x10" "0,021"
+		(property "MPN" "ERJ-3EKF1004V"
 			(at 233.68 132.08 90)
 			(hide yes)
@@
 			(project "OPC V2"
 				(path "/594181e6-a34f-458c-9685-d994528736df/e6add8e5-d5b5-453a-af59-4f27d08ef450"
-					(reference "R4")
+					(reference "R7")
 					(unit 1)
 				)
@@
 			)
 		)
-		(property "MF" "Würth Elektronik"
+		(property "px_x10" "0.031"
 			(at 184.15 107.95 0)
 			(hide yes)
@@
 			)
 		)
-		(property "px_x10" "0.031"
+		(property "MF" "Würth Elektronik"
 			(at 184.15 107.95 0)
 			(hide yes)
@@
 			)
 		)
-		(property "MPN" "TS3A4751PWR "
+		(property "px_x1" "1,49"
 			(at 175.26 137.16 0)
 			(hide yes)
@@
 			)
 		)
-		(property "px_x1" "1,49"
+		(property "px_x10" "1.09"
 			(at 175.26 137.16 0)
 			(hide yes)
@@
 			)
 		)
-		(property "px_x10" "1.09"
+		(property "MPN" "TS3A4751PWR "
 			(at 175.26 137.16 0)
 			(hide yes)
@@
 		(dnp no)
 		(fields_autoplaced yes)
-		(property "Reference" "R1"
+		(property "Reference" "R3"
 			(at 227.33 123.19 90)
 			(show_name no)
@@
 			)
 		)
-		(property "MF" "Panasonic"
+		(property "px_x1" "0,086"
 			(at 227.33 129.54 90)
 			(hide yes)
@@
 			)
 		)
-		(property "MPN" "ERJ-3EKF1004V"
+		(property "px_x10" "0.02"
 			(at 227.33 129.54 90)
 			(hide yes)
@@
 			)
 		)
-		(property "px_x1" "0,086"
+		(property "MF" "Panasonic"
 			(at 227.33 129.54 90)
 			(hide yes)
@@
 			)
 		)
-		(property "px_x10" "0,021"
+		(property "MPN" "ERJ-3EKF1004V"
 			(at 227.33 129.54 90)
 			(hide yes)
@@
 			(project "OPC V2"
 				(path "/594181e6-a34f-458c-9685-d994528736df/e6add8e5-d5b5-453a-af59-4f27d08ef450"
-					(reference "R1")
+					(reference "R3")
 					(unit 1)
 				)
@@
 			)
 		)
-		(property "MF" "Würth Elektronik"
+		(property "px_x10" "0.031"
 			(at 86.36 114.3 0)
 			(hide yes)
@@
 			)
 		)
-		(property "px_x10" "0.031"
+		(property "MF" "Würth Elektronik"
 			(at 86.36 114.3 0)
 			(hide yes)
@@
 			)
 		)
-		(property "MF" "Würth Elektronik"
+		(property "px_x10" "0.031"
 			(at 74.93 31.75 0)
 			(hide yes)
@@
 			)
 		)
-		(property "px_x10" "0.031"
+		(property "MF" "Würth Elektronik"
 			(at 74.93 31.75 0)
 			(hide yes)
@@
 		(dnp no)
 		(fields_autoplaced yes)
-		(property "Reference" "R2"
+		(property "Reference" "R5"
 			(at 220.98 120.65 90)
 			(show_name no)
@@
 			)
 		)
-		(property "MF" "Panasonic"
+		(property "px_x1" "0.619"
 			(at 220.98 127 90)
 			(hide yes)
@@
 			)
 		)
-		(property "MPN" "ERA-3ARB1652V"
+		(property "px_x10" "0,446 "
 			(at 220.98 127 90)
 			(hide yes)
@@
 			)
 		)
-		(property "px_x1" "0.619"
+		(property "MF" "Panasonic"
 			(at 220.98 127 90)
 			(hide yes)
@@
 			)
 		)
-		(property "px_x10" "0,446 "
+		(property "MPN" "ERA-3ARB1652V"
 			(at 220.98 127 90)
 			(hide yes)
@@
 			(project "OPC V2"
 				(path "/594181e6-a34f-458c-9685-d994528736df/e6add8e5-d5b5-453a-af59-4f27d08ef450"
-					(reference "R2")
+					(reference "R5")
 					(unit 1)
 				)
@@
 			)
 		)
-		(property "MF" "Würth Elektronik"
+		(property "px_x10" "0.031"
 			(at 227.33 31.75 0)
 			(hide yes)
@@
 			)
 		)
-		(property "px_x10" "0.031"
+		(property "MF" "Würth Elektronik"
 			(at 227.33 31.75 0)
 			(hide yes)
@@
 			)
 		)
-		(property "MPN" "TS3A4751PWR "
+		(property "px_x1" "1,49"
 			(at 66.04 60.96 0)
 			(hide yes)
@@
 			)
 		)
-		(property "px_x1" "1,49"
+		(property "px_x10" "1.09"
 			(at 66.04 60.96 0)
 			(hide yes)
@@
 			)
 		)
-		(property "px_x10" "1.09"
+		(property "MPN" "TS3A4751PWR "
 			(at 66.04 60.96 0)
 			(hide yes)
@@
 			)
 		)
-		(property "MF" "Würth Elektronik"
+		(property "px_x10" "0.031"
 			(at 151.13 31.75 0)
 			(hide yes)
@@
 			)
 		)
-		(property "px_x10" "0.031"
+		(property "MF" "Würth Elektronik"
 			(at 151.13 31.75 0)
 			(hide yes)
@@
 			)
 		)
-		(property "MPN" "TS3A4751PWR "
+		(property "px_x1" "1,49"
 			(at 218.44 60.96 0)
 			(hide yes)
@@
 			)
 		)
-		(property "px_x1" "1,49"
+		(property "px_x10" "1.09"
 			(at 218.44 60.96 0)
 			(hide yes)
@@
 			)
 		)
-		(property "px_x10" "1.09"
+		(property "MPN" "TS3A4751PWR "
 			(at 218.44 60.96 0)
 			(hide yes)
@@
 			)
 		)
-		(property "MPN" "TS3A4751PWR "
+		(property "px_x1" "1,49"
 			(at 77.47 143.51 0)
 			(hide yes)
@@
 			)
 		)
-		(property "px_x1" "1,49"
+		(property "px_x10" "1.09"
 			(at 77.47 143.51 0)
 			(hide yes)
@@
 			)
 		)
-		(property "px_x10" "1.09"
+		(property "MPN" "TS3A4751PWR "
 			(at 77.47 143.51 0)
 			(hide yes)
@@
 		(dnp no)
 		(fields_autoplaced yes)
-		(property "Reference" "R7"
+		(property "Reference" "R9"
 			(at 207.01 118.11 90)
 			(show_name no)
@@
 			)
 		)
-		(property "MF" "Panasonic"
+		(property "px_x1" "0.344"
 			(at 207.01 124.46 90)
 			(hide yes)
@@
 			)
 		)
-		(property "MPN" "ERA-3ARB332V"
+		(property "px_x10" "0,25"
 			(at 207.01 124.46 90)
 			(hide yes)
@@
 			)
 		)
-		(property "px_x1" "0.344"
+		(property "MF" "Panasonic"
 			(at 207.01 124.46 90)
 			(hide yes)
@@
 			)
 		)
-		(property "px_x10" "0,25"
+		(property "MPN" "ERA-3ARB332V"
 			(at 207.01 124.46 90)
 			(hide yes)
@@
 			(project "OPC V2"
 				(path "/594181e6-a34f-458c-9685-d994528736df/e6add8e5-d5b5-453a-af59-4f27d08ef450"
-					(reference "R7")
+					(reference "R9")
 					(unit 1)
 				)

Commit message: avant prod
Parts:
- R10, R9: footprint Resistor_SMD:R_0603_1608Metric_Pad0.98x0.95mm_HandSolder -> Resistor_SMD:R_0805_2012Metric; LCSC Part # (none) -> C19679588; MPN ERA-3ARB332V -> ERA-6ARB332V; px_x1 0.344 -> 0.396; px_x10 0,25 -> 0,28
- R3, R7: footprint Resistor_SMD:R_0603_1608Metric_Pad0.98x0.95mm_HandSolder -> Resistor_SMD:R_0805_2012Metric; LCSC Part # C23182 -> C17514
- R5: footprint Resistor_SMD:R_0603_1608Metric_Pad0.98x0.95mm_HandSolder -> Resistor_SMD:R_0805_2012Metric; LCSC Part # (none) -> C47115532; MPN ERA-3ARB1652V -> ERA-6ARB1652V; px_x1 0.619 -> 0.628; px_x10 0,446 -> 0,486
Other:
- note added: "R5 & R9 & R10 => Low ppm/K !"
- note removed: "R2 & R6 & R7 => Low ppm/K !"
- moved on the sheet: R5
Changed lines of the file:
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@@
 		)
 	)
-	(text "R2 & R6 & R7 => Low ppm/K !"
+	(text "R5 & R9 & R10 => Low ppm/K !"
 		(exclude_from_sim no)
 		(at 232.156 102.87 0)
@@
 	)
 	(junction
-		(at 237.49 127)
-		(diameter 0)
-		(color 0 0 0 0)
-	)
-	(junction
 		(at 81.28 60.96)
 		(diameter 0)
@@
 		(color 0 0 0 0)
 	)
+	(junction
+		(at 237.49 127)
+		(diameter 0)
+		(color 0 0 0 0)
+	)
 	(wire
 		(pts
@@
 	(wire
 		(pts
-			(xy 224.79 127) (xy 237.49 127)
+			(xy 220.98 127) (xy 237.49 127)
 		)
 		(stroke
@@
 	(wire
 		(pts
-			(xy 190.5 127) (xy 217.17 127)
+			(xy 190.5 127) (xy 213.36 127)
 		)
 		(stroke
@@
 			)
 		)
-		(property "Footprint" "Resistor_SMD:R_0603_1608Metric_Pad0.98x0.95mm_HandSolder"
+		(property "Footprint" "Resistor_SMD:R_0805_2012Metric"
 			(at 207.01 117.348 90)
 			(hide yes)
@@
 			)
 		)
-		(property "px_x1" "0.344"
+		(property "px_x1" "0.396"
 			(at 207.01 115.57 90)
 			(hide yes)
@@
 			)
 		)
-		(property "px_x10" "0,25"
+		(property "px_x10" "0,28"
 			(at 207.01 115.57 90)
 			(hide yes)
@@
 			)
 		)
-		(property "MPN" "ERA-3ARB332V"
+		(property "MPN" "ERA-6ARB332V"
+			(at 207.01 115.57 90)
+			(hide yes)
+			(show_name no)
+			(do_not_autoplace no)
+			(effects
+				(font
+					(size 1.27 1.27)
+				)
+			)
+		)
+		(property "LCSC Part #" "C19679588"
 			(at 207.01 115.57 90)
 			(hide yes)
@@
 			)
 		)
-		(property "Footprint" "Resistor_SMD:R_0603_1608Metric_Pad0.98x0.95mm_HandSolder"
+		(property "Footprint" "Resistor_SMD:R_0805_2012Metric"
 			(at 233.68 133.858 90)
 			(hide yes)
@@
 			)
 		)
-		(property "LCSC Part #" "C23182"
+		(property "LCSC Part #" "C17514"
 			(at 233.68 132.08 90)
 			(hide yes)
@@
 			)
 		)
-		(property "Footprint" "Resistor_SMD:R_0603_1608Metric_Pad0.98x0.95mm_HandSolder"
+		(property "Footprint" "Resistor_SMD:R_0805_2012Metric"
 			(at 227.33 131.318 90)
 			(hide yes)
@@
 			)
 		)
-		(property "LCSC Part #" "C23182"
+		(property "LCSC Part #" "C17514"
 			(at 227.33 129.54 90)
 			(hide yes)
@@
 	(symbol
 		(lib_id "Device:R")
-		(at 220.98 127 90)
+		(at 217.17 127 90)
 		(unit 1)
 		(body_style 1)
@@
 		(fields_autoplaced yes)
 		(property "Reference" "R5"
-			(at 220.98 120.65 90)
+			(at 217.17 120.65 90)
 			(show_name no)
 			(do_not_autoplace no)
@@
 		)
 		(property "Value" "16k5"
-			(at 220.98 123.19 90)
+			(at 217.17 123.19 90)
 			(show_name no)
 			(do_not_autoplace no)
@@
 			)
 		)
-		(property "Footprint" "Resistor_SMD:R_0603_1608Metric_Pad0.98x0.95mm_HandSolder"
-			(at 220.98 128.778 90)
+		(property "Footprint" "Resistor_SMD:R_0805_2012Metric"
+			(at 217.17 128.778 90)
 			(hide yes)
 			(show_name no)
@@
 		)
 		(property "Datasheet" "ERA-6ARB332V"
-			(at 220.98 127 0)
+			(at 217.17 127 0)
 			(hide yes)
 			(show_name no)
@@
 		)
 		(property "Description" "Resistor"
-			(at 220.98 127 0)
+			(at 217.17 127 0)
 			(hide yes)
 			(show_name no)
@@
 			)
 		)
-		(property "px_x1" "0.619"
-			(at 220.98 127 90)
+		(property "px_x1" "0.628"
+			(at 217.17 127 90)
 			(hide yes)
 			(show_name no)
@@
 			)
 		)
-		(property "px_x10" "0,446 "
-			(at 220.98 127 90)
+		(property "px_x10" "0,486"
+			(at 217.17 127 90)
 			(hide yes)
 			(show_name no)
@@
 		)
 		(property "MF" "Panasonic"
-			(at 220.98 127 90)
+			(at 217.17 127 90)
 			(hide yes)
 			(show_name no)
@@
 			)
 		)
-		(property "MPN" "ERA-3ARB1652V"
-			(at 220.98 127 90)
+		(property "MPN" "ERA-6ARB1652V"
+			(at 217.17 127 90)
+			(hide yes)
+			(show_name no)
+			(do_not_autoplace no)
+			(effects
+				(font
+					(size 1.27 1.27)
+				)
+			)
+		)
+		(property "LCSC Part #" "C47115532"
+			(at 217.17 127 90)
 			(hide yes)
 			(show_name no)
@@
 			)
 		)
-		(property "Footprint" "Resistor_SMD:R_0603_1608Metric_Pad0.98x0.95mm_HandSolder"
+		(property "Footprint" "Resistor_SMD:R_0805_2012Metric"
 			(at 207.01 126.238 90)
 			(hide yes)
@@
 			)
 		)
-		(property "px_x1" "0.344"
+		(property "px_x1" "0.396"
 			(at 207.01 124.46 90)
 			(hide yes)
@@
 			)
 		)
-		(property "px_x10" "0,25"
+		(property "px_x10" "0,28"
 			(at 207.01 124.46 90)
 			(hide yes)
@@
 			)
 		)
-		(property "MPN" "ERA-3ARB332V"
+		(property "MPN" "ERA-6ARB332V"
+			(at 207.01 124.46 90)
+			(hide yes)
+			(show_name no)
+			(do_not_autoplace no)
+			(effects
+				(font
+					(size 1.27 1.27)
+				)
+			)
+		)
+		(property "LCSC Part #" "C19679588"
 			(at 207.01 124.46 90)
 			(hide yes)

Commit message: MAJ post prod
Other:
- note added: "Inputs & mulitplexeur pour selectionner l'entrée"
- note removed: "Inputs & multiplexing"
- title: Entrées -> Entrées & Mulitplexage
Changed lines of the file:
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@@
 	(paper "A4")
 	(title_block
-		(title "Entrées")
+		(title "Entrées & Mulitplexage")
+		(date "2026-08-17")
+		(rev "0.2")
 	)
 	(rectangle
@@
 		)
 	)
-	(text "Inputs & multiplexing"
+	(text "Inputs & mulitplexeur pour selectionner l'entrée"
 		(exclude_from_sim no)
 		(at 143.002 16.256 0)
@@
 		)
 		(instances
-			(project "OPC V2"
+			(project "OPC V3"
 				(path "/594181e6-a34f-458c-9685-d994528736df/e6add8e5-d5b5-453a-af59-4f27d08ef450"
 					(reference "U6")
@@
 		)
 		(instances
-			(project "OPC V2"
+			(project "OPC V3"
 				(path "/594181e6-a34f-458c-9685-d994528736df/e6add8e5-d5b5-453a-af59-4f27d08ef450"
 					(reference "R10")
@@
 		)
 		(instances
-			(project "OPC V2"
+			(project "OPC V3"
 				(path "/594181e6-a34f-458c-9685-d994528736df/e6add8e5-d5b5-453a-af59-4f27d08ef450"
 					(reference "#PWR066")
@@
 		)
 		(instances
-			(project "OPC V2"
+			(project "OPC V3"
 				(path "/594181e6-a34f-458c-9685-d994528736df/e6add8e5-d5b5-453a-af59-4f27d08ef450"
 					(reference "#PWR08")
@@
 		)
 		(instances
-			(project "OPC V2"
+			(project "OPC V3"
 				(path "/594181e6-a34f-458c-9685-d994528736df/e6add8e5-d5b5-453a-af59-4f27d08ef450"
 					(reference "#PWR04")
@@
 		)
 		(instances
-			(project "OPC V2"
+			(project "OPC V3"
 				(path "/594181e6-a34f-458c-9685-d994528736df/e6add8e5-d5b5-453a-af59-4f27d08ef450"
 					(reference "#PWR011")
@@
 		)
 		(instances
-			(project "OPC V2"
+			(project "OPC V3"
 				(path "/594181e6-a34f-458c-9685-d994528736df/e6add8e5-d5b5-453a-af59-4f27d08ef450"
 					(reference "#PWR05")
@@
 		)
 		(instances
-			(project "OPC V2"
+			(project "OPC V3"
 				(path "/594181e6-a34f-458c-9685-d994528736df/e6add8e5-d5b5-453a-af59-4f27d08ef450"
 					(reference "R7")
@@
 		)
 		(instances
-			(project "OPC V2"
+			(project "OPC V3"
 				(path "/594181e6-a34f-458c-9685-d994528736df/e6add8e5-d5b5-453a-af59-4f27d08ef450"
 					(reference "#PWR012")
@@
 		)
 		(instances
-			(project "OPC V2"
+			(project "OPC V3"
 				(path "/594181e6-a34f-458c-9685-d994528736df/e6add8e5-d5b5-453a-af59-4f27d08ef450"
 					(reference "#PWR010")
@@
 		)
 		(instances
-			(project "OPC V2"
+			(project "OPC V3"
 				(path "/594181e6-a34f-458c-9685-d994528736df/e6add8e5-d5b5-453a-af59-4f27d08ef450"
 					(reference "C7")
@@
 		)
 		(instances
-			(project "OPC V2"
+			(project "OPC V3"
 				(path "/594181e6-a34f-458c-9685-d994528736df/e6add8e5-d5b5-453a-af59-4f27d08ef450"
 					(reference "#PWR06")
@@
 		)
 		(instances
-			(project "OPC V2"
+			(project "OPC V3"
 				(path "/594181e6-a34f-458c-9685-d994528736df/e6add8e5-d5b5-453a-af59-4f27d08ef450"
 					(reference "#PWR061")
@@
 		)
 		(instances
-			(project "OPC V2"
+			(project "OPC V3"
 				(path "/594181e6-a34f-458c-9685-d994528736df/e6add8e5-d5b5-453a-af59-4f27d08ef450"
 					(reference "U4")
@@
 		)
 		(instances
-			(project "OPC V2"
+			(project "OPC V3"
 				(path "/594181e6-a34f-458c-9685-d994528736df/e6add8e5-d5b5-453a-af59-4f27d08ef450"
 					(reference "R3")
@@
 		)
 		(instances
-			(project "OPC V2"
+			(project "OPC V3"
 				(path "/594181e6-a34f-458c-9685-d994528736df/e6add8e5-d5b5-453a-af59-4f27d08ef450"
 					(reference "C3")
@@
 		)
 		(instances
-			(project "OPC V2"
+			(project "OPC V3"
 				(path "/594181e6-a34f-458c-9685-d994528736df/e6add8e5-d5b5-453a-af59-4f27d08ef450"
 					(reference "C2")
@@
 		)
 		(instances
-			(project "OPC V2"
+			(project "OPC V3"
 				(path "/594181e6-a34f-458c-9685-d994528736df/e6add8e5-d5b5-453a-af59-4f27d08ef450"
 					(reference "R5")
@@
 		)
 		(instances
-			(project "OPC V2"
+			(project "OPC V3"
 				(path "/594181e6-a34f-458c-9685-d994528736df/e6add8e5-d5b5-453a-af59-4f27d08ef450"
 					(reference "#PWR07")
@@
 		)
 		(instances
-			(project "OPC V2"
+			(project "OPC V3"
 				(path "/594181e6-a34f-458c-9685-d994528736df/e6add8e5-d5b5-453a-af59-4f27d08ef450"
 					(reference "#PWR016")
@@
 		)
 		(instances
-			(project "OPC V2"
+			(project "OPC V3"
 				(path "/594181e6-a34f-458c-9685-d994528736df/e6add8e5-d5b5-453a-af59-4f27d08ef450"
 					(reference "#PWR03")
@@
 		)
 		(instances
-			(project "OPC V2"
+			(project "OPC V3"
 				(path "/594181e6-a34f-458c-9685-d994528736df/e6add8e5-d5b5-453a-af59-4f27d08ef450"
 					(reference "#PWR013")
@@
 		)
 		(instances
-			(project "OPC V2"
+			(project "OPC V3"
 				(path "/594181e6-a34f-458c-9685-d994528736df/e6add8e5-d5b5-453a-af59-4f27d08ef450"
 					(reference "#PWR09")
@@
 		)
 		(instances
-			(project "OPC V2"
+			(project "OPC V3"
 				(path "/594181e6-a34f-458c-9685-d994528736df/e6add8e5-d5b5-453a-af59-4f27d08ef450"
 					(reference "#PWR01")
@@
 		)
 		(instances
-			(project "OPC V2"
+			(project "OPC V3"
 				(path "/594181e6-a34f-458c-9685-d994528736df/e6add8e5-d5b5-453a-af59-4f27d08ef450"
 					(reference "J4")
@@
 		)
 		(instances
-			(project "OPC V2"
+			(project "OPC V3"
 				(path "/594181e6-a34f-458c-9685-d994528736df/e6add8e5-d5b5-453a-af59-4f27d08ef450"
 					(reference "#PWR02")
@@
 		)
 		(instances
-			(project "OPC V2"
+			(project "OPC V3"
 				(path "/594181e6-a34f-458c-9685-d994528736df/e6add8e5-d5b5-453a-af59-4f27d08ef450"
 					(reference "#PWR015")
@@
 		)
 		(instances
-			(project "OPC V2"
+			(project "OPC V3"
 				(path "/594181e6-a34f-458c-9685-d994528736df/e6add8e5-d5b5-453a-af59-4f27d08ef450"
 					(reference "C11")
@@
 		)
 		(instances
-			(project "OPC V2"
+			(project "OPC V3"
 				(path "/594181e6-a34f-458c-9685-d994528736df/e6add8e5-d5b5-453a-af59-4f27d08ef450"
 					(reference "J1")
@@
 		)
 		(instances
-			(project "OPC V2"
+			(project "OPC V3"
 				(path "/594181e6-a34f-458c-9685-d994528736df/e6add8e5-d5b5-453a-af59-4f27d08ef450"
 					(reference "U2")
@@
 		)
 		(instances
-			(project "OPC V2"
+			(project "OPC V3"
 				(path "/594181e6-a34f-458c-9685-d994528736df/e6add8e5-d5b5-453a-af59-4f27d08ef450"
 					(reference "C8")
@@
 		)
 		(instances
-			(project "OPC V2"
+			(project "OPC V3"
 				(path "/594181e6-a34f-458c-9685-d994528736df/e6add8e5-d5b5-453a-af59-4f27d08ef450"
 					(reference "#PWR014")
@@
 		)
 		(instances
-			(project "OPC V2"
+			(project "OPC V3"
 				(path "/594181e6-a34f-458c-9685-d994528736df/e6add8e5-d5b5-453a-af59-4f27d08ef450"
 					(reference "U9")
@@
 		)
 		(instances
-			(project "OPC V2"
+			(project "OPC V3"
 				(path "/594181e6-a34f-458c-9685-d994528736df/e6add8e5-d5b5-453a-af59-4f27d08ef450"
 					(reference "J2")
@@
 		)
 		(instances
-			(project "OPC V2"
+			(project "OPC V3"
 				(path "/594181e6-a34f-458c-9685-d994528736df/e6add8e5-d5b5-453a-af59-4f27d08ef450"
 					(reference "U1")
@@
 		)
 		(instances
-			(project "OPC V2"
+			(project "OPC V3"
 				(path "/594181e6-a34f-458c-9685-d994528736df/e6add8e5-d5b5-453a-af59-4f27d08ef450"
 					(reference "R9")
