File: pEntrees.kicad_sch (KiCad schematic)
At the start: 16 parts, among them U8 ISO1212

Commit message: corrections
Parts:
- renumbered C14 to C3, C13 to C6, C24 to C7, D4 to D10, D5 to D11, R18 to R1, R15 to R2, R14 to R3, R17 to R4, R12 to R5, R13 to R6, RV1 to RV10, RV2 to RV11, U8 to U2
Changed lines of the file:
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@@
 		(dnp no)
 		(fields_autoplaced yes)
-		(property "Reference" "RV1"
+		(property "Reference" "RV10"
 			(at 82.55 80.2032 0)
 			(hide yes)
@@
 			(project "puissance"
 				(path "/b2e6993f-467e-4b42-9c79-23dbe0260143/97bef727-136c-4ae9-bc19-a701a61b21b2"
-					(reference "RV1")
+					(reference "RV10")
 					(unit 1)
 				)
@@
 		(in_pos_files yes)
 		(dnp no)
-		(property "Reference" "R15"
+		(property "Reference" "R2"
 			(at 135.89 91.44 90)
 			(show_name no)
@@
 			(project "puissance"
 				(path "/b2e6993f-467e-4b42-9c79-23dbe0260143/97bef727-136c-4ae9-bc19-a701a61b21b2"
-					(reference "R15")
+					(reference "R2")
 					(unit 1)
 				)
@@
 		(in_pos_files yes)
 		(dnp no)
-		(property "Reference" "C13"
+		(property "Reference" "C6"
 			(at 102.87 80.0162 0)
 			(show_name no)
@@
 			(project "puissance"
 				(path "/b2e6993f-467e-4b42-9c79-23dbe0260143/97bef727-136c-4ae9-bc19-a701a61b21b2"
-					(reference "C13")
+					(reference "C6")
 					(unit 1)
 				)
@@
 		(dnp no)
 		(fields_autoplaced yes)
-		(property "Reference" "R17"
+		(property "Reference" "R4"
 			(at 120.65 80.0099 0)
 			(show_name no)
@@
 			(project "puissance"
 				(path "/b2e6993f-467e-4b42-9c79-23dbe0260143/97bef727-136c-4ae9-bc19-a701a61b21b2"
-					(reference "R17")
+					(reference "R4")
 					(unit 1)
 				)
@@
 		(dnp no)
 		(fields_autoplaced yes)
-		(property "Reference" "D5"
+		(property "Reference" "D11"
 			(at 93.98 105.4099 90)
 			(hide yes)
@@
 			(project "puissance"
 				(path "/b2e6993f-467e-4b42-9c79-23dbe0260143/97bef727-136c-4ae9-bc19-a701a61b21b2"
-					(reference "D5")
+					(reference "D11")
 					(unit 1)
 				)
@@
 		(dnp no)
 		(fields_autoplaced yes)
-		(property "Reference" "R18"
+		(property "Reference" "R1"
 			(at 120.65 101.5999 0)
 			(show_name no)
@@
 			(project "puissance"
 				(path "/b2e6993f-467e-4b42-9c79-23dbe0260143/97bef727-136c-4ae9-bc19-a701a61b21b2"
-					(reference "R18")
+					(reference "R1")
 					(unit 1)
 				)
@@
 		(in_pos_files yes)
 		(dnp no)
-		(property "Reference" "C24"
+		(property "Reference" "C7"
 			(at 173.99 62.2362 0)
 			(show_name no)
@@
 			(project "puissance"
 				(path "/b2e6993f-467e-4b42-9c79-23dbe0260143/97bef727-136c-4ae9-bc19-a701a61b21b2"
-					(reference "C24")
+					(reference "C7")
 					(unit 1)
 				)
@@
 		(in_pos_files yes)
 		(dnp no)
-		(property "Reference" "R14"
+		(property "Reference" "R3"
 			(at 101.6 88.9 90)
 			(show_name no)
@@
 			(project "puissance"
 				(path "/b2e6993f-467e-4b42-9c79-23dbe0260143/97bef727-136c-4ae9-bc19-a701a61b21b2"
-					(reference "R14")
+					(reference "R3")
 					(unit 1)
 				)
@@
 		(dnp no)
 		(fields_autoplaced yes)
-		(property "Reference" "D4"
+		(property "Reference" "D10"
 			(at 93.98 81.2799 90)
 			(hide yes)
@@
 			(project "puissance"
 				(path "/b2e6993f-467e-4b42-9c79-23dbe0260143/97bef727-136c-4ae9-bc19-a701a61b21b2"
-					(reference "D4")
+					(reference "D10")
 					(unit 1)
 				)
@@
 		(dnp no)
 		(fields_autoplaced yes)
-		(property "Reference" "U8"
+		(property "Reference" "U2"
 			(at 168.5133 74.93 0)
 			(show_name no)
@@
 			(project "puissance"
 				(path "/b2e6993f-467e-4b42-9c79-23dbe0260143/97bef727-136c-4ae9-bc19-a701a61b21b2"
-					(reference "U8")
+					(reference "U2")
 					(unit 1)
 				)
@@
 		(dnp no)
 		(fields_autoplaced yes)
-		(property "Reference" "R13"
+		(property "Reference" "R6"
 			(at 101.6 67.31 90)
 			(show_name no)
@@
 			(project "puissance"
 				(path "/b2e6993f-467e-4b42-9c79-23dbe0260143/97bef727-136c-4ae9-bc19-a701a61b21b2"
-					(reference "R13")
+					(reference "R6")
 					(unit 1)
 				)
@@
 		(dnp no)
 		(fields_autoplaced yes)
-		(property "Reference" "R12"
+		(property "Reference" "R5"
 			(at 135.89 78.74 90)
 			(show_name no)
@@
 			(project "puissance"
 				(path "/b2e6993f-467e-4b42-9c79-23dbe0260143/97bef727-136c-4ae9-bc19-a701a61b21b2"
-					(reference "R12")
+					(reference "R5")
 					(unit 1)
 				)
@@
 		(in_pos_files yes)
 		(dnp no)
-		(property "Reference" "C14"
+		(property "Reference" "C3"
 			(at 102.87 104.1462 0)
 			(show_name no)
@@
 			(project "puissance"
 				(path "/b2e6993f-467e-4b42-9c79-23dbe0260143/97bef727-136c-4ae9-bc19-a701a61b21b2"
-					(reference "C14")
+					(reference "C3")
 					(unit 1)
 				)
@@
 		(dnp no)
 		(fields_autoplaced yes)
-		(property "Reference" "RV2"
+		(property "Reference" "RV11"
 			(at 82.55 104.3332 0)
 			(hide yes)
@@
 			(project "puissance"
 				(path "/b2e6993f-467e-4b42-9c79-23dbe0260143/97bef727-136c-4ae9-bc19-a701a61b21b2"
-					(reference "RV2")
-					(unit 1)
-				)
+					(reference "RV11")
+					(unit 1)
+				)

Commit message: daily
Parts:
- D10, D11, RV10, RV11: now left out of the parts list
- R2, R5: LCSC Part # C336827 -> C23204
- R3, R6: LCSC Part # C22940 -> C17526

Commit message: daily
Parts:
- C3, C6: value 10n -> 10n 100V; MPN (none) -> GRM188R72A103MA01J; px_1 (none) -> 0.086; px_10 (none) -> 0.02
- C7: value 0.1µ -> 0.1µ 10V; MF (none) -> Würth Elektronik; MPN (none) -> 885012206020; px_1 (none) -> 0,095; px_10 (none) -> 0.031
- R1, R4: now left out of the parts list
- R2, R5: MPN (none) -> ERJ-3GEYJ560V; px_1 (none) -> 0.086; px_10 (none) -> 0.02
- R3, R6: MPN (none) -> ERJ-6GEYJ242V; px_1 (none) -> 0.086; px_10 (none) -> 0.025
- U2: MPN (none) -> ISO1212DBQR; px_1 (none) -> 1.14; px_10 (none) -> 0.828

Commit message: avant prod
Parts:
- R3, R6: value 2k4 -> 1000; footprint Resistor_SMD:R_0805_2012Metric_Pad1.20x1.40mm_HandSolder -> Resistor_SMD:R_1206_3216Metric; LCSC Part # C17526 -> C4410
Connections:
- net Input1: now also R6.1; no longer R3.1
- net Input2: now also R3.1; no longer R6.1
Other:
- note added: "Changer la valeur de R6 et cliquer sur le tableau"
- note added: "TP1 & TP2 sont là pour la dissipation de chaleur"
- note added: "Tension de seuil de détection du signal"
- note added: "Vin (max) = @{60 + ${/b2e6993f-467e-4b42-9c79-23dbe0260143/97bef727-136c-4ae9-bc19-a701a61b21b2/99e0dbed-f0a7-4f4c-9860-5a011a33f80f:VALUE} * 0.0021 * 562 / ${/b2e6993f-467e-4b42-9c79-23dbe0260143/97bef727-136c-4ae9-bc19-a701a61b21b2/c8e65150-a29e-4934-ab6e-f5d5b94ba4d4:VALUE}}V"
- moved on the sheet: TP1

Commit message: MAJ post prod
Other:
- title: (none) -> Entreés numériques
Changed lines of the file:
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@@
 	(generator_version "10.0")
 	(paper "A4")
+	(title_block
+		(title "Entreés numériques")
+		(date "2026-08-17")
+		(rev "0.2")
+	)
 	(rectangle
 		(start 59.69 39.37)
