File: pSorties_sch.kicad_sch (KiCad schematic)
At the start: 20 parts, among them K5 G6DN-1A-L DC24, K6 G6DN-1A-L DC24, U12 PDRV81545PWPR, U13 ISO6420FDR, U14 TLV75709PDBV

Commit message: corrections
Parts:
- added C10, C9: 0.1µ, Capacitor_SMD:C_0603_1608Metric_Pad1.08x0.95mm_HandSolder, symbol Device:C_Small
- added Q2, Q3: 2N7002, PCM_Package_TO_SOT_SMD_AKL:SOT-23, symbol PCM_Transistor_MOSFET_AKL:2N7002
- added R10, R12: 47k, Resistor_SMD:R_0603_1608Metric_Pad0.98x0.95mm_HandSolder, symbol Device:R
- added R11, R13: 470, Resistor_SMD:R_0603_1608Metric_Pad0.98x0.95mm_HandSolder, symbol Device:R
- U3: renamed from U12; value PDRV81545PWPR -> DRV81545PWPR
- U5: renamed from U14; value TLV75709PDBV -> TLV709
- renumbered C19 to C11, C20 to C12, C22 to C14, C21 to C15, C1 to C5, C23 to C8, D8 to D2, D7 to D3, D6 to D4, K5 to K1, K6 to K2, OC2 to OC1, R16 to R7, R24 to R8, R23 to R9, RV4 to RV1, RV3 to RV2, U13 to U4
Connections:
- net +3V3: now also C9.1
- net GND1: now also C9.2
- net GND2: now also C10.2, Q2.2 (S), Q3.2 (S), R10.1, R12.1; no longer OC1.5, OC1.7
- net at D3.2 (A), K1.A1: now also Q3.3 (D); no longer OC1.6
- net at D4.2 (A), K2.A1: now also Q2.3 (D); no longer OC1.8
- net +5VP: now reaches C12.1, U4.8 (VCC2), U5.5 (OUT)
- net +5VP: now also OC1.6, OC1.8, C10.1
- new net: Q3.1 (G), R12.2, R13.2
- new net: OC1.5, R13.1
- new net: OC1.7, R11.1
- new net: Q2.1 (G), R10.2, R11.2

Commit message: daily
Parts:
- C12: value 0.47µ -> 1µ; LCSC Part # C1623 -> C15849
- C5: LCSC Part # C14663 -> C72523
- U5: value TLV709 -> TLV709A50DBVR
- renumbered D2 to D3, D3 to D4, D4 to D5, Q3 to Q1, R8 to R10, R9 to R11, R10 to R12, R11 to R13, R12 to R8, R13 to R9
Changed lines of the file:
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@@
 		(in_pos_files yes)
 		(dnp no)
-		(property "Reference" "R9"
+		(property "Reference" "R11"
 			(at 219.71 123.19 90)
 			(show_name no)
@@
 			(project "puissance"
 				(path "/b2e6993f-467e-4b42-9c79-23dbe0260143/39db9153-1d42-494d-ad76-9efc4a0a86d2"
-					(reference "R9")
+					(reference "R11")
 					(unit 1)
 				)
@@
 		(in_pos_files yes)
 		(dnp no)
-		(property "Reference" "Q3"
+		(property "Reference" "Q1"
 			(at 165.1 140.9699 0)
 			(show_name no)
@@
 			(project "puissance"
 				(path "/b2e6993f-467e-4b42-9c79-23dbe0260143/39db9153-1d42-494d-ad76-9efc4a0a86d2"
-					(reference "Q3")
+					(reference "Q1")
 					(unit 1)
 				)
@@
 		(in_pos_files yes)
 		(dnp no)
-		(property "Reference" "R13"
+		(property "Reference" "R9"
 			(at 193.0399 146.05 0)
 			(show_name no)
@@
 			(project "puissance"
 				(path "/b2e6993f-467e-4b42-9c79-23dbe0260143/39db9153-1d42-494d-ad76-9efc4a0a86d2"
-					(reference "R13")
+					(reference "R9")
 					(unit 1)
 				)
@@
 		(in_pos_files yes)
 		(dnp no)
-		(property "Reference" "D2"
+		(property "Reference" "D3"
 			(at 100.3301 53.34 90)
 			(show_name no)
@@
 			(project "puissance"
 				(path "/b2e6993f-467e-4b42-9c79-23dbe0260143/39db9153-1d42-494d-ad76-9efc4a0a86d2"
-					(reference "D2")
+					(reference "D3")
 					(unit 1)
 				)
@@
 		(in_pos_files yes)
 		(dnp no)
-		(property "Reference" "R11"
+		(property "Reference" "R13"
 			(at 195.58 126.9999 0)
 			(show_name no)
@@
 			(project "puissance"
 				(path "/b2e6993f-467e-4b42-9c79-23dbe0260143/39db9153-1d42-494d-ad76-9efc4a0a86d2"
-					(reference "R11")
+					(reference "R13")
 					(unit 1)
 				)
@@
 		(dnp no)
 		(fields_autoplaced yes)
-		(property "Reference" "D4"
+		(property "Reference" "D5"
 			(at 144.78 121.9199 90)
 			(show_name no)
@@
 			(project "puissance"
 				(path "/b2e6993f-467e-4b42-9c79-23dbe0260143/39db9153-1d42-494d-ad76-9efc4a0a86d2"
-					(reference "D4")
+					(reference "D5")
 					(unit 1)
 				)
@@
 			)
 		)
-		(property "Value" "0.47µ"
+		(property "Value" "1µ"
 			(at 184.658 39.37 0)
 			(show_name no)
@@
 			)
 		)
-		(property "LCSC Part #" "C1623"
+		(property "LCSC Part #" "C15849"
 			(at 180.34 39.37 0)
 			(hide yes)
@@
 		(dnp no)
 		(fields_autoplaced yes)
-		(property "Reference" "D3"
+		(property "Reference" "D4"
 			(at 144.78 143.5099 90)
 			(show_name no)
@@
 			(project "puissance"
 				(path "/b2e6993f-467e-4b42-9c79-23dbe0260143/39db9153-1d42-494d-ad76-9efc4a0a86d2"
-					(reference "D3")
+					(reference "D4")
 					(unit 1)
 				)
@@
 			)
 		)
-		(property "Value" "TLV709"
+		(property "Value" "TLV709A50DBVR"
 			(at 172.72 30.48 0)
 			(show_name no)
@@
 			)
 		)
-		(property "Datasheet" "Fixed 5V"
+		(property "Datasheet" ""
 			(at 172.72 35.56 0)
 			(hide yes)
@@
 			)
 		)
-		(property "Description" "1A Low IQ Small Size Low Dropout Voltage Regulator, Fixed Output 0.9V, SOT-23-5"
+		(property "Description" "LDO 5V"
 			(at 172.72 36.83 0)
 			(hide yes)
@@
 			)
 		)
-		(property "LCSC Part #" "C14663"
+		(property "LCSC Part #" "C72523"
 			(at 121.92 40.64 0)
 			(hide yes)
@@
 		(in_pos_files yes)
 		(dnp no)
-		(property "Reference" "R10"
+		(property "Reference" "R12"
 			(at 184.15 126.9999 0)
 			(show_name no)
@@
 			(project "puissance"
 				(path "/b2e6993f-467e-4b42-9c79-23dbe0260143/39db9153-1d42-494d-ad76-9efc4a0a86d2"
-					(reference "R10")
+					(reference "R12")
 					(unit 1)
 				)
@@
 		(in_pos_files yes)
 		(dnp no)
-		(property "Reference" "R12"
+		(property "Reference" "R8"
 			(at 184.15 146.0499 0)
 			(show_name no)
@@
 			(project "puissance"
 				(path "/b2e6993f-467e-4b42-9c79-23dbe0260143/39db9153-1d42-494d-ad76-9efc4a0a86d2"
-					(reference "R12")
+					(reference "R8")
 					(unit 1)
 				)
@@
 		(in_pos_files yes)
 		(dnp no)
-		(property "Reference" "R8"
+		(property "Reference" "R10"
 			(at 229.87 132.08 90)
 			(show_name no)
@@
 			(project "puissance"
 				(path "/b2e6993f-467e-4b42-9c79-23dbe0260143/39db9153-1d42-494d-ad76-9efc4a0a86d2"
-					(reference "R8")
+					(reference "R10")
 					(unit 1)
 				)

Commit message: daily
Parts:
- added JP1: SolderJumper_2_Open, Jumper:SolderJumper-2_P1.3mm_Open_RoundedPad1.0x1.5mm, symbol Jumper:SolderJumper_2_Open
- C10, C9: value 0.1µ -> 0.1µ 10V; MF (none) -> Würth Elektronik; MPN (none) -> 885012206020; px_1 (none) -> 0,095; px_10 (none) -> 0.031
- C11: value 0.1µ -> 0.1µ 50V; MPN (none) -> GCM188L81H104MA57D; px_1 (none) -> 0,095; px_10 (none) -> 0.035
- C12, C8: value 1µ -> 1µ 50V; footprint Capacitor_SMD:C_0603_1608Metric_Pad1.08x0.95mm_HandSolder -> Capacitor_SMD:C_0805_2012Metric_Pad1.18x1.45mm_HandSolder; LCSC Part # C15849 -> C28323; MF (none) -> Murata; MPN (none) -> GRM219R61H105MA73D; px_1 (none) -> 0.129; px_10 (none) -> 0.052
- C14, C15: value 10n -> 10n 100V; footprint Capacitor_SMD:C_0805_2012Metric_Pad1.18x1.45mm_HandSolder -> Capacitor_SMD:C_0603_1608Metric_Pad1.08x0.95mm_HandSolder; LCSC Part # C1710 -> C57112; MPN (none) -> GRM188R72A103MA01J; px_1 (none) -> 0.086; px_10 (none) -> 0.02
- C5: MPN (none) -> 865080645012; px_1 (none) -> 0,292; px_10 (none) -> 0.287
- D3: MPN (none) -> 824501331; px_1 (none) -> 0,318; px_10 (none) -> 0.297
- D4, D5: value US1M -> FR1G; MPN (none) -> FR1G; px_1 (none) -> 0,095; px_10 (none) -> 0.066
- K1, K2: MPN (none) -> G6DN-1A-L DC24; px_1 (none) -> 2,42; px_10 (none) -> 2.22
- OC1: MPN (none) -> MOCD217M; px_1 (none) -> 0,869; px_10 (none) -> .573
- Q1, Q2: MF (none) -> Toshiba; MPN (none) -> T2N7002BK,LM
- R10, R11: MPN (none) -> ERJ-3GEYJ152V; px_1 (none) -> 0.086; px_10 (none) -> 0.02
- R12, R8: MPN (none) -> ERJ-3GEYJ473V; px_1 (none) -> 0.086; px_10 (none) -> 0.02
- R13, R9: MPN (none) -> ERJ-3GEYJ470V; px_1 (none) -> 0.086; px_10 (none) -> 0.02
- R7: MPN (none) -> ERJ-3GEYJ333V; px_1 (none) -> 0.086; px_10 (none) -> 0.02
- RV1, RV2: MF (none) -> Bourns; MPN (none) -> MOV-07D391KKTR; px_1 (none) -> 0.129; px_10 (none) -> 0.078
- U3: MPN (none) -> DRV81545PWPR; px_1 (none) -> 2.43; px_10 (none) -> 1.81
- U4: MPN (none) -> ISO6420FDR; px_1 (none) -> 1.26; px_10 (none) -> 0.92
- U5: MPN (none) -> TLV709A50DBVR; px_1 (none) -> 0.499; px_10 (none) -> 0.352
Connections:
- net +24V: now also JP1.2 (B)
- net at D3.1 (K), U3.18 (VCLAMP), U3.3 (VCLAMP): now also JP1.1 (A)
Other:
- moved on the sheet: D3

Commit message: avant prod
Parts:
- OC1: LCSC Part # (none) -> C258262
- Q1, Q2: LCSC Part # (none) -> C8545
- U3: LCSC Part # (none) -> C53201928
Connections:
- net Output1: now also C15.1, U3.16 (OUT2), U3.17 (OUT1); no longer C14.1, U3.14 (OUT4), U3.15 (OUT3)
- net Output2: now also C14.1, U3.14 (OUT4), U3.15 (OUT3); no longer C15.1, U3.16 (OUT2), U3.17 (OUT1)
Other:
- note added: "Imax = 5 A (250 VAC or 30 VDC)"
- note added: "Voutput (max) = 55V Si Voutput > 24VDC -> Adapter la TVS Si Voutput = Vin (24VDC) -> Possiblité de shunter la TVS mais il faut souder le jumper C14 & C15 Faculatif (ESD filtering)"
- moved on the sheet: C14, C15
Changed lines of the file:
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@@
 	(paper "A4")
 	(rectangle
-		(start 62.23 21.59)
+		(start 33.02 21.59)
 		(end 256.54 99.06)
 		(stroke
@@
 	)
 	(rectangle
-		(start 62.23 107.95)
+		(start 33.02 107.95)
 		(end 256.54 161.29)
 		(stroke
@@
 		)
 	)
+	(text "Voutput (max) = 55V\n\nSi Voutput > 24VDC \n	-> Adapter la TVS\n\nSi Voutput = Vin (24VDC)\n	-> Possiblité de shunter la TVS mais il faut souder le jumper\n\nC14 & C15 Faculatif (ESD filtering)"
+		(exclude_from_sim no)
+		(at 34.036 23.622 0)
+		(effects
+			(font
+				(size 1.27 1.27)
+			)
+			(justify left top)
+		)
+	)
+	(text "Imax =  5 A (250 VAC or 30 VDC)"
+		(exclude_from_sim no)
+		(at 37.084 113.03 0)
+		(effects
+			(font
+				(size 1.27 1.27)
+			)
+			(justify left top)
+		)
+	)
 	(text "Sorties logiques"
 		(exclude_from_sim no)
@@
 	)
 	(junction
-		(at 106.68 68.58)
-		(diameter 0)
-		(color 0 0 0 0)
-	)
-	(junction
 		(at 146.05 63.5)
 		(diameter 0)
@@
 	)
 	(junction
-		(at 99.06 63.5)
+		(at 186.69 152.4)
 		(diameter 0)
 		(color 0 0 0 0)
 	)
 	(junction
-		(at 106.68 91.44)
+		(at 142.24 135.89)
 		(diameter 0)
 		(color 0 0 0 0)
 	)
 	(junction
-		(at 186.69 152.4)
+		(at 104.14 68.58)
 		(diameter 0)
 		(color 0 0 0 0)
 	)
 	(junction
-		(at 142.24 135.89)
+		(at 135.89 151.13)
 		(diameter 0)
 		(color 0 0 0 0)
 	)
 	(junction
-		(at 135.89 151.13)
+		(at 142.24 114.3)
 		(diameter 0)
 		(color 0 0 0 0)
 	)
 	(junction
-		(at 142.24 114.3)
+		(at 146.05 91.44)
 		(diameter 0)
 		(color 0 0 0 0)
 	)
 	(junction
-		(at 146.05 91.44)
+		(at 91.44 63.5)
 		(diameter 0)
 		(color 0 0 0 0)
@@
 	)
 	(junction
+		(at 104.14 91.44)
+		(diameter 0)
+		(color 0 0 0 0)
+	)
+	(junction
 		(at 153.67 91.44)
 		(diameter 0)
@@
 	(wire
 		(pts
-			(xy 106.68 91.44) (xy 110.49 91.44)
-		)
-		(stroke
-			(width 0)
-			(type default)
-		)
-	)
-	(wire
-		(pts
 			(xy 198.12 66.04) (xy 189.23 66.04)
 		)
@@
 	(wire
 		(pts
-			(xy 106.68 81.28) (xy 106.68 91.44)
+			(xy 104.14 81.28) (xy 104.14 91.44)
 		)
 		(stroke
@@
 	(wire
 		(pts
-			(xy 73.66 63.5) (xy 99.06 63.5)
+			(xy 73.66 63.5) (xy 91.44 63.5)
 		)
 		(stroke
@@
 	(wire
 		(pts
+			(xy 104.14 68.58) (xy 110.49 68.58)
+		)
+		(stroke
+			(width 0)
+			(type default)
+		)
+	)
+	(wire
+		(pts
 			(xy 142.24 125.73) (xy 142.24 129.54)
 		)
@@
 	(wire
 		(pts
-			(xy 99.06 63.5) (xy 99.06 71.12)
+			(xy 91.44 63.5) (xy 91.44 71.12)
 		)
 		(stroke
@@
 	(wire
 		(pts
-			(xy 106.68 68.58) (xy 106.68 76.2)
+			(xy 104.14 68.58) (xy 104.14 76.2)
 		)
 		(stroke
@@
 	(wire
 		(pts
-			(xy 99.06 91.44) (xy 106.68 91.44)
+			(xy 91.44 91.44) (xy 104.14 91.44)
 		)
 		(stroke
@@
 	(wire
 		(pts
-			(xy 73.66 68.58) (xy 106.68 68.58)
+			(xy 73.66 68.58) (xy 104.14 68.58)
 		)
 		(stroke
@@
 	(wire
 		(pts
+			(xy 91.44 63.5) (xy 110.49 63.5)
+		)
+		(stroke
+			(width 0)
+			(type default)
+		)
+	)
+	(wire
+		(pts
 			(xy 85.09 132.08) (xy 107.95 132.08)
 		)
@@
 	(wire
 		(pts
+			(xy 104.14 91.44) (xy 110.49 91.44)
+		)
+		(stroke
+			(width 0)
+			(type default)
+		)
+	)
+	(wire
+		(pts
 			(xy 130.81 114.3) (xy 142.24 114.3)
 		)
@@
 	(wire
 		(pts
-			(xy 99.06 76.2) (xy 99.06 91.44)
+			(xy 91.44 76.2) (xy 91.44 91.44)
 		)
 		(stroke
@@
 	(wire
 		(pts
-			(xy 106.68 68.58) (xy 110.49 68.58)
-		)
-		(stroke
-			(width 0)
-			(type default)
-		)
-	)
-	(wire
-		(pts
 			(xy 218.44 45.72) (xy 218.44 46.99)
 		)
@@
 	(wire
 		(pts
-			(xy 99.06 63.5) (xy 110.49 63.5)
-		)
-		(stroke
-			(width 0)
-			(type default)
-		)
-	)
-	(wire
-		(pts
 			(xy 194.31 46.99) (xy 194.31 58.42)
 		)
@@
 		)
 	)
-	(hierarchical_label "Output1"
+	(hierarchical_label "Output2"
 		(shape output)
 		(at 73.66 68.58 180)
@@
 		)
 	)
-	(hierarchical_label "Output2"
+	(hierarchical_label "Output1"
 		(shape output)
 		(at 73.66 63.5 180)
@@
 			)
 		)
+		(property "LCSC Part #" "C8545"
+			(at 171.45 142.24 0)
+			(hide yes)
+			(show_name no)
+			(do_not_autoplace no)
+			(effects
+				(font
+					(size 1.27 1.27)
+				)
+			)
+		)
 		(pin "3"
 		)
@@
 			)
 		)
+		(property "LCSC Part #" "C258262"
+			(at 208.28 132.08 0)
+			(hide yes)
+			(show_name no)
+			(do_not_autoplace no)
+			(effects
+				(font
+					(size 1.27 1.27)
+				)
+			)
+		)
 		(pin "1"
 		)
@@
 	(symbol
 		(lib_id "Device:C_Small")
-		(at 99.06 73.66 0)
+		(at 91.44 73.66 0)
 		(mirror y)
 		(unit 1)
@@
 		(dnp no)
 		(property "Reference" "C15"
-			(at 96.52 72.3962 0)
+			(at 88.9 72.3962 0)
 			(show_name no)
 			(do_not_autoplace no)
@@
 		)
 		(property "Value" "10n 100V"
-			(at 96.52 74.9362 0)
+			(at 88.9 74.9362 0)
 			(show_name no)
 			(do_not_autoplace no)
@@
 		)
 		(property "Footprint" "Capacitor_SMD:C_0603_1608Metric_Pad1.08x0.95mm_HandSolder"
-			(at 99.06 73.66 0)
+			(at 91.44 73.66 0)
 			(hide yes)
 			(show_name no)
@@
 		)
 		(property "Datasheet" "GCM188R71H104KA57D"
-			(at 99.06 73.66 0)
+			(at 91.44 73.66 0)
 			(hide yes)
 			(show_name no)
@@
 		)
 		(property "Description" "Unpolarized capacitor, small symbol"
-			(at 99.06 73.66 0)
+			(at 91.44 73.66 0)
 			(hide yes)
 			(show_name no)
@@
 		)
 		(property "LCSC Part #" "C57112"
-			(at 99.06 73.66 0)
+			(at 91.44 73.66 0)
 			(hide yes)
 			(show_name no)
@@
 		)
 		(property "px_1" "0.086"
-			(at 99.06 73.66 0)
+			(at 91.44 73.66 0)
 			(hide yes)
 			(show_name no)
@@
 		)
 		(property "px_10" "0.02"
-			(at 99.06 73.66 0)
+			(at 91.44 73.66 0)
 			(hide yes)
 			(show_name no)
@@
 		)
 		(property "MPN" "GRM188R72A103MA01J"
-			(at 99.06 73.66 0)
+			(at 91.44 73.66 0)
 			(hide yes)
 			(show_name no)
@@
 			)
 		)
-		(property "Datasheet" ""
+		(property "Datasheet" "https://omronfs.omron.com/en_US/ecb/products/pdf/en-g6dn.pdf"
 			(at 125.73 121.92 0)
 			(hide yes)
@@
 			)
 		)
+		(property "LCSC Part #" "C53201928"
+			(at 128.27 68.58 0)
+			(hide yes)
+			(show_name no)
+			(do_not_autoplace no)
+			(effects
+				(font
+					(size 1.27 1.27)
+				)
+			)
+		)
 		(pin "17"
 		)
@@
 	(symbol
 		(lib_id "Device:C_Small")
-		(at 106.68 78.74 0)
+		(at 104.14 78.74 0)
 		(mirror y)
 		(unit 1)
@@
 		(dnp no)
 		(property "Reference" "C14"
-			(at 104.14 77.4762 0)
+			(at 101.6 77.4762 0)
 			(show_name no)
 			(do_not_autoplace no)
@@
 		)
 		(property "Value" "10n 100V"
-			(at 104.14 80.0162 0)
+			(at 101.6 80.0162 0)
 			(show_name no)
 			(do_not_autoplace no)
@@
 		)
 		(property "Footprint" "Capacitor_SMD:C_0603_1608Metric_Pad1.08x0.95mm_HandSolder"
-			(at 106.68 78.74 0)
+			(at 104.14 78.74 0)
 			(hide yes)
 			(show_name no)
@@
 		)
 		(property "Datasheet" "GCM188R71H104KA57D"
-			(at 106.68 78.74 0)
+			(at 104.14 78.74 0)
 			(hide yes)
 			(show_name no)
@@
 		)
 		(property "Description" "Unpolarized capacitor, small symbol"
-			(at 106.68 78.74 0)
+			(at 104.14 78.74 0)
 			(hide yes)
 			(show_name no)
@@
 		)
 		(property "LCSC Part #" "C57112"
-			(at 106.68 78.74 0)
+			(at 104.14 78.74 0)
 			(hide yes)
 			(show_name no)
@@
 		)
 		(property "px_1" "0.086"
-			(at 106.68 78.74 0)
+			(at 104.14 78.74 0)
 			(hide yes)
 			(show_name no)
@@
 		)
 		(property "px_10" "0.02"
-			(at 106.68 78.74 0)
+			(at 104.14 78.74 0)
 			(hide yes)
 			(show_name no)
@@
 		)
 		(property "MPN" "GRM188R72A103MA01J"
-			(at 106.68 78.74 0)
+			(at 104.14 78.74 0)
 			(hide yes)
 			(show_name no)
@@
 			)
 		)
+		(property "LCSC Part #" "C8545"
+			(at 181.61 119.38 0)
+			(hide yes)
+			(show_name no)
+			(do_not_autoplace no)
+			(effects
+				(font
+					(size 1.27 1.27)
+				)
+			)
+		)
 		(pin "3"
 		)
@@
 			)
 		)
-		(property "Datasheet" ""
+		(property "Datasheet" "https://omronfs.omron.com/en_US/ecb/products/pdf/en-g6dn.pdf"
 			(at 125.73 143.51 0)
 			(hide yes)

Commit message: MAJ post prod
Other:
- title: (none) -> Sorties PWM & Relais
Changed lines of the file:
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@@
 	(generator_version "10.0")
 	(paper "A4")
+	(title_block
+		(title "Sorties PWM & Relais")
+		(date "2026-08-17")
+		(rev "0.2")
+	)
 	(rectangle
 		(start 33.02 21.59)
