File: pico.kicad_sch (KiCad schematic)
At the start: 20 parts, among them J5 Conn_01x05, J6 Conn_01x04_Pin, U3 MCP23017x-x-ML, U7 BMP581, U8 DS3231MZ

Commit message: pre prod
Parts:
- RN1, RN2, RN3: LCSC Part # (none) -> C29718
Changed lines of the file:
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@@
+			)
+		)
+		(property "LCSC Part #" "C29718"
+			(at 168.91 97.79 0)
+			(hide yes)
+			(show_name no)
+			(do_not_autoplace no)
+			(effects
+				(font
+					(size 1.27 1.27)
+				)
 			)
 		)
@@
 			)
 		)
+		(property "LCSC Part #" "C29718"
+			(at 140.97 97.79 0)
+			(hide yes)
+			(show_name no)
+			(do_not_autoplace no)
+			(effects
+				(font
+					(size 1.27 1.27)
+				)
+			)
+		)
 		(pin "4"
 		)
@@
 			(at 156.21 97.79 0)
 			(hide yes)
+			(show_name no)
+			(do_not_autoplace no)
+			(effects
+				(font
+					(size 1.27 1.27)
+				)
+			)
+		)
+		(property "LCSC Part #" "C29718"
+			(at 156.21 97.79 0)
+			(hide yes)

Commit message: MAJ post prod
Other:
- note added: "GPIO expansion pull-down"
- note removed: "GPIO explansion pull-down"
Changed lines of the file:
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@@
 	(title_block
 		(title "Microcontroleur & GPIO")
+		(date "2026-08-17")
+		(rev "0.2")
 	)
 	(rectangle
@@
 		)
 	)
-	(text "GPIO explansion pull-down"
+	(text "GPIO expansion pull-down"
 		(exclude_from_sim no)
 		(at 159.512 55.372 0)
@@
 		)
 		(instances
-			(project "OPC V2"
+			(project "OPC V3"
 				(path "/594181e6-a34f-458c-9685-d994528736df/1471a511-d5fc-4a40-8bcc-7e3684e303d6"
 					(reference "#PWR026")
@@
 		)
 		(instances
-			(project "OPC V2"
+			(project "OPC V3"
 				(path "/594181e6-a34f-458c-9685-d994528736df/1471a511-d5fc-4a40-8bcc-7e3684e303d6"
 					(reference "#PWR027")
@@
 		)
 		(instances
-			(project "OPC V2"
+			(project "OPC V3"
 				(path "/594181e6-a34f-458c-9685-d994528736df/1471a511-d5fc-4a40-8bcc-7e3684e303d6"
 					(reference "C10")
@@
 		)
 		(instances
-			(project "OPC V2"
+			(project "OPC V3"
 				(path "/594181e6-a34f-458c-9685-d994528736df/1471a511-d5fc-4a40-8bcc-7e3684e303d6"
 					(reference "D1")
@@
 		)
 		(instances
-			(project "OPC V2"
+			(project "OPC V3"
 				(path "/594181e6-a34f-458c-9685-d994528736df/1471a511-d5fc-4a40-8bcc-7e3684e303d6"
 					(reference "R2")
@@
 		(dnp no)
 		(property "Reference" "A1"
-			(at 72.644 71.628 0)
+			(at 73.406 50.546 0)
 			(show_name no)
 			(do_not_autoplace no)
@@
 		)
 		(instances
-			(project "OPC V2"
+			(project "OPC V3"
 				(path "/594181e6-a34f-458c-9685-d994528736df/1471a511-d5fc-4a40-8bcc-7e3684e303d6"
 					(reference "A1")
@@
 		)
 		(instances
-			(project "OPC V2"
+			(project "OPC V3"
 				(path "/594181e6-a34f-458c-9685-d994528736df/1471a511-d5fc-4a40-8bcc-7e3684e303d6"
 					(reference "RN2")
@@
 		)
 		(instances
-			(project "OPC V2"
+			(project "OPC V3"
 				(path "/594181e6-a34f-458c-9685-d994528736df/1471a511-d5fc-4a40-8bcc-7e3684e303d6"
 					(reference "#PWR050")
@@
 		)
 		(instances
-			(project "OPC V2"
+			(project "OPC V3"
 				(path "/594181e6-a34f-458c-9685-d994528736df/1471a511-d5fc-4a40-8bcc-7e3684e303d6"
 					(reference "#PWR042")
@@
 		)
 		(instances
-			(project "OPC V2"
+			(project "OPC V3"
 				(path "/594181e6-a34f-458c-9685-d994528736df/1471a511-d5fc-4a40-8bcc-7e3684e303d6"
 					(reference "R12")
@@
 		)
 		(instances
-			(project "OPC V2"
+			(project "OPC V3"
 				(path "/594181e6-a34f-458c-9685-d994528736df/1471a511-d5fc-4a40-8bcc-7e3684e303d6"
 					(reference "#PWR040")
@@
 		)
 		(instances
-			(project "OPC V2"
+			(project "OPC V3"
 				(path "/594181e6-a34f-458c-9685-d994528736df/1471a511-d5fc-4a40-8bcc-7e3684e303d6"
 					(reference "#PWR043")
@@
 		)
 		(instances
-			(project "OPC V2"
+			(project "OPC V3"
 				(path "/594181e6-a34f-458c-9685-d994528736df/1471a511-d5fc-4a40-8bcc-7e3684e303d6"
 					(reference "#PWR045")
@@
 		)
 		(instances
-			(project "OPC V2"
+			(project "OPC V3"
 				(path "/594181e6-a34f-458c-9685-d994528736df/1471a511-d5fc-4a40-8bcc-7e3684e303d6"
 					(reference "#PWR037")
@@
 		)
 		(instances
-			(project "OPC V2"
+			(project "OPC V3"
 				(path "/594181e6-a34f-458c-9685-d994528736df/1471a511-d5fc-4a40-8bcc-7e3684e303d6"
 					(reference "C9")
@@
 		)
 		(instances
-			(project "OPC V2"
+			(project "OPC V3"
 				(path "/594181e6-a34f-458c-9685-d994528736df/1471a511-d5fc-4a40-8bcc-7e3684e303d6"
 					(reference "#PWR029")
@@
 		)
 		(instances
-			(project "OPC V2"
+			(project "OPC V3"
 				(path "/594181e6-a34f-458c-9685-d994528736df/1471a511-d5fc-4a40-8bcc-7e3684e303d6"
 					(reference "RN3")
@@
 		)
 		(instances
-			(project "OPC V2"
+			(project "OPC V3"
 				(path "/594181e6-a34f-458c-9685-d994528736df/1471a511-d5fc-4a40-8bcc-7e3684e303d6"
 					(reference "#PWR046")
@@
 		)
 		(instances
-			(project "OPC V2"
+			(project "OPC V3"
 				(path "/594181e6-a34f-458c-9685-d994528736df/1471a511-d5fc-4a40-8bcc-7e3684e303d6"
 					(reference "#PWR028")
@@
 		)
 		(instances
-			(project "OPC V2"
+			(project "OPC V3"
 				(path "/594181e6-a34f-458c-9685-d994528736df/1471a511-d5fc-4a40-8bcc-7e3684e303d6"
 					(reference "U8")
@@
 		)
 		(instances
-			(project "OPC V2"
+			(project "OPC V3"
 				(path "/594181e6-a34f-458c-9685-d994528736df/1471a511-d5fc-4a40-8bcc-7e3684e303d6"
 					(reference "D2")
@@
 		)
 		(instances
-			(project "OPC V2"
+			(project "OPC V3"
 				(path "/594181e6-a34f-458c-9685-d994528736df/1471a511-d5fc-4a40-8bcc-7e3684e303d6"
 					(reference "R14")
@@
 		)
 		(instances
-			(project "OPC V2"
+			(project "OPC V3"
 				(path "/594181e6-a34f-458c-9685-d994528736df/1471a511-d5fc-4a40-8bcc-7e3684e303d6"
 					(reference "#PWR032")
@@
 		)
 		(instances
-			(project "OPC V2"
+			(project "OPC V3"
 				(path "/594181e6-a34f-458c-9685-d994528736df/1471a511-d5fc-4a40-8bcc-7e3684e303d6"
 					(reference "#PWR078")
@@
 		)
 		(instances
-			(project "OPC V2"
+			(project "OPC V3"
 				(path "/594181e6-a34f-458c-9685-d994528736df/1471a511-d5fc-4a40-8bcc-7e3684e303d6"
 					(reference "C6")
@@
 		)
 		(instances
-			(project "OPC V2"
+			(project "OPC V3"
 				(path "/594181e6-a34f-458c-9685-d994528736df/1471a511-d5fc-4a40-8bcc-7e3684e303d6"
 					(reference "RN1")
@@
 		(dnp no)
 		(property "Reference" "U3"
-			(at 228.092 45.212 0)
+			(at 227.076 40.386 0)
 			(show_name no)
 			(do_not_autoplace no)
@@
 		)
 		(property "Value" "MCP23017x-x-ML"
-			(at 215.392 57.912 0)
+			(at 212.344 42.926 0)
 			(show_name no)
 			(do_not_autoplace no)
@@
 		)
 		(instances
-			(project "OPC V2"
+			(project "OPC V3"
 				(path "/594181e6-a34f-458c-9685-d994528736df/1471a511-d5fc-4a40-8bcc-7e3684e303d6"
 					(reference "U3")
@@
 		)
 		(instances
-			(project "OPC V2"
+			(project "OPC V3"
 				(path "/594181e6-a34f-458c-9685-d994528736df/1471a511-d5fc-4a40-8bcc-7e3684e303d6"
 					(reference "#PWR051")
@@
 		)
 		(instances
-			(project "OPC V2"
+			(project "OPC V3"
 				(path "/594181e6-a34f-458c-9685-d994528736df/1471a511-d5fc-4a40-8bcc-7e3684e303d6"
 					(reference "#PWR048")
@@
 		)
 		(instances
-			(project "OPC V2"
+			(project "OPC V3"
 				(path "/594181e6-a34f-458c-9685-d994528736df/1471a511-d5fc-4a40-8bcc-7e3684e303d6"
 					(reference "J5")
@@
 		)
 		(instances
-			(project "OPC V2"
+			(project "OPC V3"
 				(path "/594181e6-a34f-458c-9685-d994528736df/1471a511-d5fc-4a40-8bcc-7e3684e303d6"
 					(reference "U7")
@@
 		)
 		(instances
-			(project "OPC V2"
+			(project "OPC V3"
 				(path "/594181e6-a34f-458c-9685-d994528736df/1471a511-d5fc-4a40-8bcc-7e3684e303d6"
 					(reference "#PWR039")
@@
 		)
 		(instances
-			(project "OPC V2"
+			(project "OPC V3"
 				(path "/594181e6-a34f-458c-9685-d994528736df/1471a511-d5fc-4a40-8bcc-7e3684e303d6"
 					(reference "J6")
@@
 		)
 		(instances
-			(project "OPC V2"
+			(project "OPC V3"
 				(path "/594181e6-a34f-458c-9685-d994528736df/1471a511-d5fc-4a40-8bcc-7e3684e303d6"
 					(reference "C1")
@@
 		)
 		(instances
-			(project "OPC V2"
+			(project "OPC V3"
 				(path "/594181e6-a34f-458c-9685-d994528736df/1471a511-d5fc-4a40-8bcc-7e3684e303d6"
 					(reference "#PWR044")
@@
 		)
 		(instances
-			(project "OPC V2"
+			(project "OPC V3"
 				(path "/594181e6-a34f-458c-9685-d994528736df/1471a511-d5fc-4a40-8bcc-7e3684e303d6"
 					(reference "#PWR047")
@@
 		)
 		(instances
-			(project "OPC V2"
+			(project "OPC V3"
 				(path "/594181e6-a34f-458c-9685-d994528736df/1471a511-d5fc-4a40-8bcc-7e3684e303d6"
 					(reference "#PWR030")
@@
 		)
 		(instances
-			(project "OPC V2"
+			(project "OPC V3"
 				(path "/594181e6-a34f-458c-9685-d994528736df/1471a511-d5fc-4a40-8bcc-7e3684e303d6"
 					(reference "#PWR036")
@@
 		)
 		(instances
-			(project "OPC V2"
+			(project "OPC V3"
 				(path "/594181e6-a34f-458c-9685-d994528736df/1471a511-d5fc-4a40-8bcc-7e3684e303d6"
 					(reference "R13")
@@
 		)
 		(instances
-			(project "OPC V2"
+			(project "OPC V3"
 				(path "/594181e6-a34f-458c-9685-d994528736df/1471a511-d5fc-4a40-8bcc-7e3684e303d6"
 					(reference "#PWR041")
@@
 		)
 		(instances
-			(project "OPC V2"
+			(project "OPC V3"
 				(path "/594181e6-a34f-458c-9685-d994528736df/1471a511-d5fc-4a40-8bcc-7e3684e303d6"
 					(reference "#PWR038")
@@
 		)
 		(instances
-			(project "OPC V2"
+			(project "OPC V3"
 				(path "/594181e6-a34f-458c-9685-d994528736df/1471a511-d5fc-4a40-8bcc-7e3684e303d6"
 					(reference "C12")
@@
 		)
 		(instances
-			(project "OPC V2"
+			(project "OPC V3"
 				(path "/594181e6-a34f-458c-9685-d994528736df/1471a511-d5fc-4a40-8bcc-7e3684e303d6"
 					(reference "#PWR049")
