File: puissance.kicad_sch (KiCad schematic)
At the start: 41 parts, among them J5 Screw_Terminal_01x10, J8 MEC1-110-02-F-D-A, J9 Screw_Terminal_01x04, K5 G6DN-1A-L DC24, K6 G6DN-1A-L DC24, U11 SIP-4_1779205311, U12 PDRV81545PWPR, U13 ISO7720D, U14 TLV75709PDBV, U8 ISO1212

Commit message: update
Connections:
- net Input1_MCU: now also J8.17
- net Input2_MCU: now also J8.19
- net Output1_MCU: now also J8.11
- net Output2_MCU: now also J8.15
- net Relay1_MCU: now also J8.07
- net Relay2_MCU: now also J8.09

Commit message: suite et nouvel écran
Parts:
- removed C13, C14, C19: 0.1µ, Capacitor_SMD:C_0603_1608Metric_Pad1.08x0.95mm_HandSolder, symbol Device:C_Small
- removed C20: 0.47µ, Capacitor_SMD:C_0603_1608Metric_Pad1.08x0.95mm_HandSolder, symbol Device:C_Small
- removed C21, C22: 10n, Capacitor_SMD:C_0805_2012Metric_Pad1.18x1.45mm_HandSolder, symbol Device:C_Small
- removed D4, D5: (no value), symbol PCM_Diode_TVS_AKL:D_TVS_Bidirectional_Generic
- removed D6, D7: US1M, Diode_SMD:D_SMA, symbol Device:D
- removed D8: SMAJ33CA, PCM_Diode_SMD_AKL:D_SMA_TVS, symbol PCM_Diode_TVS_AKL:SMAJ33CA
- removed J9: Screw_Terminal_01x04, TerminalBlock_Phoenix:TerminalBlock_Phoenix_MPT-0,5-4-2.54_1x04_P2.54mm_Horizontal, symbol Connector:Screw_Terminal_01x04
- removed K5, K6: G6DN-1A-L DC24, OPC:G6DN, symbol Relay:Relay_SPST-NO
- removed OC2: MOCD217M, PCM_Package_SO_AKL:SO-8_3.9x6.2mm_P1.27mm, symbol PCM_Optocoupler_AKL:ILD213T
- removed R12, R15: 562, Resistor_SMD:R_0603_1608Metric_Pad0.98x0.95mm_HandSolder, symbol Device:R
- removed R13, R14: 2k5, Resistor_SMD:R_0603_1608Metric_Pad0.98x0.95mm_HandSolder, symbol Device:R
- removed R16: 33k, Resistor_SMD:R_0603_1608Metric_Pad0.98x0.95mm_HandSolder, symbol Device:R
- removed R23, R24: 1k5, Resistor_SMD:R_0603_1608Metric_Pad0.98x0.95mm_HandSolder, symbol Device:R
- removed RV1, RV2: Varistor, symbol Device:Varistor
- removed RV3, RV4: MOV-07D391KKTR, Varistor:RV_Disc_D9mm_W3.9mm_P5mm, symbol Device:Varistor
- removed TP1, TP2: TestPoint, TestPoint:TestPoint_Pad_2.0x2.0mm, symbol Connector:TestPoint
- removed U12: PDRV81545PWPR, OPC:U_TSSOP_PWP0020AC_TEX, symbol OPC:PDRV81545PWPR
- removed U13: ISO7720D, Package_SO:SOIC-8_3.9x4.9mm_P1.27mm, symbol Isolator:ISO7720D
- removed U14: TLV75709PDBV, Package_TO_SOT_SMD:SOT-23-5, symbol Regulator_Linear:TLV75709PDBV
- removed U8: ISO1212, Package_SO:SSOP-16_3.9x4.9mm_P0.635mm, symbol Isolator:ISO1212
- added F1: 100mA, Fuse:Fuse_1812_4532Metric, symbol Device:Fuse
- added J2: Screw_Terminal_01x04, TerminalBlock_Phoenix:TerminalBlock_Phoenix_PT-1,5-4-3.5-H_1x04_P3.50mm_Horizontal, symbol Connector:Screw_Terminal_01x04
Connections:
- net Output1_MCU is gone; now on net Output_4: J8.11
- net Output2_MCU is gone; now on net Output_3: J8.15
- net Relay1_MCU is gone; now on net Output_6: J8.07
- net Relay2_MCU is gone; now on net Output_5: J8.09
- net +24V: now also F1.2; no longer D3.1 (K)
- net Input1_MCU: no longer J8.17
- net Input2_MCU: no longer J8.19
- net Output_6: now reaches J8.08
- net Output_5: now reaches J8.10
- net Output_4: now reaches J8.12
- net Output_3: now reaches J8.16
- net Output_2: now reaches J8.18
- net Output_2: now also J8.17
- net Output_1: now reaches J8.20
- net Output_1: now also J8.19
- net Input1 renamed Entrée/Input1
- net Input2 renamed Entrée/Input2
- net Output1 renamed Sorties/Output2
- net Output2 renamed Sorties/Output1
- net Voutput: no longer names the net of J5.10 (Pin_10)
- new net: D3.1 (K), F1.1
- new net Sorties/Relais1_COM: J2.3 (Pin_3)
- new net Sorties/Relais1_NO: J2.4 (Pin_4)
- new net Sorties/Relais2_COM: J2.1 (Pin_1)
- new net Sorties/Relais2_NO: J2.2 (Pin_2)
Other:
- added sheet Entrée (pEntrees.kicad_sch)
- added sheet Sorties (pSorties_sch.kicad_sch)
- note added: "Output 5&6 can also be used as UART or I2C UART1 master TX : 5 UART1 master RX : 6 I2C0 master sda : 5 I2C0 master sck : 6"
- note removed: "Entrées logiques"
- note removed: "OU"
- note removed: "Sorties TOR / Relais"
- note removed: "Sorties logiques"
- moved on the sheet: C15, C16, C17, C18, D3, J5, L1, U11

Commit message: corrections
Parts:
- added D5: SMAJ33CA, PCM_Diode_SMD_AKL:D_SMA_TVS, symbol PCM_Diode_TVS_AKL:SMAJ33CA
- J3: renamed from J8; now left out of the parts list
- renumbered C16 to C1, C18 to C13, C15 to C2, C17 to C4, D3 to D1, J5 to J1, U11 to U1
Connections:
- net +24V: now also D5.1 (K)
- net GND2: now also C13.2, J1.10 (Pin_10), J1.8 (Pin_8), D5.2 (A); no longer J1.7 (Pin_7)
- net Sorties/Output1: now also J1.7 (Pin_7); no longer J1.8 (Pin_8)
- net at C2.1, L1.2, U1.2 (+VIN): no longer C13.2
Other:
- moved on the sheet: C13

Commit message: daily
Parts:
- F1: footprint Fuse:Fuse_1812_4532Metric -> Fuse:Fuse_1210_3225Metric
- renumbered D5 to D2
Connections:
- net Output_1: no longer J3.19
- net Output_2: no longer J3.17
- net Output_3: no longer J3.16
- net Output_4: no longer J3.12
- net Output_5: no longer J3.10
- net Output_6: no longer J3.08
Changed lines of the file:
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@@
 	)
 	(junction
-		(at 140.97 46.99)
-		(diameter 0)
-		(color 0 0 0 0)
-	)
-	(junction
-		(at 140.97 52.07)
-		(diameter 0)
-		(color 0 0 0 0)
-	)
-	(junction
-		(at 260.35 127)
+		(at 142.24 46.99)
 		(diameter 0)
 		(color 0 0 0 0)
@@
 	)
 	(junction
-		(at 234.95 139.7)
-		(diameter 0)
-		(color 0 0 0 0)
-	)
-	(junction
-		(at 260.35 132.08)
-		(diameter 0)
-		(color 0 0 0 0)
-	)
-	(junction
-		(at 260.35 129.54)
-		(diameter 0)
-		(color 0 0 0 0)
-	)
-	(junction
-		(at 260.35 137.16)
-		(diameter 0)
-		(color 0 0 0 0)
-	)
-	(junction
 		(at 114.3 41.91)
-		(diameter 0)
-		(color 0 0 0 0)
-	)
-	(junction
-		(at 234.95 142.24)
-		(diameter 0)
-		(color 0 0 0 0)
-	)
-	(junction
-		(at 260.35 139.7)
 		(diameter 0)
 		(color 0 0 0 0)
@@
 	)
 	(junction
-		(at 260.35 142.24)
+		(at 142.24 52.07)
 		(diameter 0)
 		(color 0 0 0 0)
@@
 	(wire
 		(pts
-			(xy 234.95 139.7) (xy 260.35 139.7)
-		)
-		(stroke
-			(width 0)
-			(type default)
-		)
-	)
-	(wire
-		(pts
 			(xy 25.4 82.55) (xy 27.94 82.55)
 		)
@@
 	(wire
 		(pts
-			(xy 129.54 52.07) (xy 140.97 52.07)
+			(xy 129.54 52.07) (xy 142.24 52.07)
+		)
+		(stroke
+			(width 0)
+			(type default)
+		)
+	)
+	(wire
+		(pts
+			(xy 231.14 129.54) (xy 234.95 129.54)
 		)
 		(stroke
@@
 	(wire
 		(pts
-			(xy 264.16 132.08) (xy 260.35 132.08)
-		)
-		(stroke
-			(width 0)
-			(type default)
-		)
-	)
-	(wire
-		(pts
 			(xy 25.4 90.17) (xy 31.75 90.17)
 		)
@@
 	(wire
 		(pts
+			(xy 231.14 132.08) (xy 234.95 132.08)
+		)
+		(stroke
+			(width 0)
+			(type default)
+		)
+	)
+	(wire
+		(pts
 			(xy 262.89 116.84) (xy 262.89 119.38)
 		)
@@
 	(wire
 		(pts
-			(xy 264.16 137.16) (xy 260.35 137.16)
-		)
-		(stroke
-			(width 0)
-			(type default)
-		)
-	)
-	(wire
-		(pts
-			(xy 137.16 46.99) (xy 140.97 46.99)
+			(xy 137.16 46.99) (xy 142.24 46.99)
 		)
 		(stroke
@@
 	(wire
 		(pts
-			(xy 264.16 129.54) (xy 260.35 129.54)
-		)
-		(stroke
-			(width 0)
-			(type default)
-		)
-	)
-	(wire
-		(pts
 			(xy 25.4 72.39) (xy 27.94 72.39)
 		)
@@
 	(wire
 		(pts
-			(xy 140.97 46.99) (xy 142.24 46.99)
-		)
-		(stroke
-			(width 0)
-			(type default)
-		)
-	)
-	(wire
-		(pts
 			(xy 50.8 33.02) (xy 57.15 33.02)
 		)
@@
 	(wire
 		(pts
-			(xy 234.95 132.08) (xy 260.35 132.08)
-		)
-		(stroke
-			(width 0)
-			(type default)
-		)
-	)
-	(wire
-		(pts
 			(xy 64.77 83.82) (xy 67.31 83.82)
 		)
@@
 	(wire
 		(pts
-			(xy 234.95 127) (xy 260.35 127)
-		)
-		(stroke
-			(width 0)
-			(type default)
-		)
-	)
-	(wire
-		(pts
-			(xy 185.42 142.24) (xy 234.95 142.24)
-		)
-		(stroke
-			(width 0)
-			(type default)
-		)
-	)
-	(wire
-		(pts
-			(xy 234.95 129.54) (xy 260.35 129.54)
-		)
-		(stroke
-			(width 0)
-			(type default)
-		)
-	)
-	(wire
-		(pts
 			(xy 147.32 41.91) (xy 142.24 41.91)
 		)
@@
 	(wire
 		(pts
-			(xy 264.16 127) (xy 260.35 127)
+			(xy 231.14 127) (xy 234.95 127)
 		)
 		(stroke
@@
 	(wire
 		(pts
-			(xy 140.97 52.07) (xy 140.97 54.61)
+			(xy 142.24 52.07) (xy 142.24 54.61)
 		)
 		(stroke
@@
 	(wire
 		(pts
-			(xy 234.95 137.16) (xy 260.35 137.16)
-		)
-		(stroke
-			(width 0)
-			(type default)
-		)
-	)
-	(wire
-		(pts
-			(xy 234.95 142.24) (xy 260.35 142.24)
+			(xy 231.14 137.16) (xy 234.95 137.16)
+		)
+		(stroke
+			(width 0)
+			(type default)
+		)
+	)
+	(wire
+		(pts
+			(xy 193.04 139.7) (xy 185.42 139.7)
+		)
+		(stroke
+			(width 0)
+			(type default)
+		)
+	)
+	(wire
+		(pts
+			(xy 96.52 52.07) (xy 96.52 46.99)
 		)
 		(stroke
@@
 	(wire
 		(pts
-			(xy 140.97 46.99) (xy 140.97 52.07)
+			(xy 142.24 46.99) (xy 142.24 52.07)
 		)
 		(stroke
@@
 	(wire
 		(pts
+			(xy 193.04 142.24) (xy 185.42 142.24)
+		)
+		(stroke
+			(width 0)
+			(type default)
+		)
+	)
+	(wire
+		(pts
 			(xy 114.3 52.07) (xy 124.46 52.07)
 		)
@@
 	(wire
 		(pts
-			(xy 185.42 139.7) (xy 234.95 139.7)
-		)
-		(stroke
-			(width 0)
-			(type default)
-		)
-	)
-	(wire
-		(pts
 			(xy 185.42 134.62) (xy 193.04 134.62)
 		)
@@
 	(wire
 		(pts
-			(xy 96.52 46.99) (xy 114.3 46.99)
+			(xy 96.52 52.07) (xy 114.3 52.07)
 		)
 		(stroke
@@
 	)
 	(label "Output_5"
-		(at 264.16 129.54 0)
+		(at 231.14 129.54 180)
 		(effects
 			(font
 				(size 1.27 1.27)
 			)
-			(justify left bottom)
+			(justify right bottom)
 		)
 	)
 	(label "Output_6"
-		(at 264.16 127 0)
+		(at 231.14 127 180)
 		(effects
 			(font
 				(size 1.27 1.27)
 			)
-			(justify left bottom)
+			(justify right bottom)
 		)
 	)
@@
 		)
 	)
+	(label "Output_1"
+		(at 193.04 142.24 0)
+		(effects
+			(font
+				(size 1.27 1.27)
+			)
+			(justify left bottom)
+		)
+	)
 	(label "Output_5"
 		(at 193.04 77.47 0)
@@
 	)
 	(label "Output_4"
-		(at 264.16 132.08 0)
+		(at 231.14 132.08 180)
 		(effects
 			(font
 				(size 1.27 1.27)
 			)
-			(justify left bottom)
+			(justify right bottom)
 		)
 	)
 	(label "Output_3"
-		(at 264.16 137.16 0)
+		(at 231.14 137.16 180)
+		(effects
+			(font
+				(size 1.27 1.27)
+			)
+			(justify right bottom)
+		)
+	)
+	(label "Output_2"
+		(at 193.04 139.7 0)
 		(effects
 			(font
@@
 			)
 		)
-		(property "Datasheet" "GCM188R71H104KA57D"
+		(property "Datasheet" ""
 			(at 127 52.07 0)
 			(hide yes)
@@
 		(in_pos_files yes)
 		(dnp no)
-		(property "Reference" "D5"
+		(property "Reference" "D2"
 			(at 73.66 36.8299 90)
 			(show_name no)
@@
 			(project "puissance"
 				(path "/b2e6993f-467e-4b42-9c79-23dbe0260143"
-					(reference "D5")
+					(reference "D2")
 					(unit 1)
 				)
@@
 			)
 		)
-		(property "Footprint" "Fuse:Fuse_1812_4532Metric"
+		(property "Footprint" "Fuse:Fuse_1210_3225Metric"
 			(at 68.58 34.798 90)
 			(hide yes)
@@
 	(symbol
 		(lib_id "power:GND1")
-		(at 140.97 54.61 0)
+		(at 142.24 54.61 0)
 		(unit 1)
 		(body_style 1)
@@
 		(fields_autoplaced yes)
 		(property "Reference" "#PWR055"
-			(at 140.97 60.96 0)
+			(at 142.24 60.96 0)
 			(hide yes)
 			(show_name no)
@@
 		)
 		(property "Value" "GND1"
-			(at 140.97 59.69 0)
+			(at 142.24 59.69 0)
 			(show_name no)
 			(do_not_autoplace no)
@@
 		)
 		(property "Footprint" ""
-			(at 140.97 54.61 0)
+			(at 142.24 54.61 0)
 			(hide yes)
 			(show_name no)
@@
 		)
 		(property "Datasheet" ""
-			(at 140.97 54.61 0)
+			(at 142.24 54.61 0)
 			(hide yes)
 			(show_name no)
@@
 		)
 		(property "Description" "Power symbol creates a global label with name \"GND1\" , ground"
-			(at 140.97 54.61 0)
-			(hide yes)
-			(show_name no)
+			(at 142.24 54.61 0)
+			(hide yes)
+			(show_name no)

Commit message: daily
Parts:
- removed J1: Screw_Terminal_01x10, TerminalBlock_Phoenix:TerminalBlock_Phoenix_MPT-0,5-10-2.54_1x10_P2.54mm_Horizontal, symbol Connector:Screw_Terminal_01x10
- removed J2: Screw_Terminal_01x04, TerminalBlock_Phoenix:TerminalBlock_Phoenix_PT-1,5-4-3.5-H_1x04_P3.50mm_Horizontal, symbol Connector:Screw_Terminal_01x04
- added J4: 1705566, 1705566, symbol OPC:1705566
- added J5, J6: 1725672, 1725672, symbol OPC:1725672
- C1, C2: MPN (none) -> GRM319R61H475KA12D; px_1 (none) -> 0.206; px_10 (none) -> 0,084
- C13: MPN (none) -> 885342208024; px_1 (none) -> 0,198; px_10 (none) -> 0.116
- C4: MPN (none) -> GRM188R61A106ME69D; px_1 (none) -> 0,103; px_10 (none) -> 0.04
- D1: value US1M -> FR1G; MPN (none) -> FR1G; px_1 (none) -> 0,095; px_10 (none) -> 0.066
- D2: MPN (none) -> 824501331; px_1 (none) -> 0,318; px_10 (none) -> 0.297
- F1: MPN (none) -> 0ZCH0010FF2E; px_1 (none) -> 0,155; px_10 (none) -> 0.114
- L1: MF (none) -> Taiyo yuden; MPN (none) -> MAMK2520T1R0M; px_1 (none) -> 0,138; px_10 (none) -> 0.112
- U1: MPN (none) -> 1779205311; px_1 (none) -> 2.73; px_10 (none) -> 2.51
Connections:
- net Entrée/Input1: now also J6.3
- net Entrée/Input2: now also J6.4
- net GND2: now also J5.2, J5.4, J6.2
- net Sorties/Output1: now also J5.1
- net Sorties/Output2: now also J5.3
- net Sorties/Relais1_COM: now also J4.5 (3.1), J4.6 (3.2)
- net Sorties/Relais1_NO: now also J4.7 (4.1), J4.8 (4.2)
- net Sorties/Relais2_COM: now also J4.1 (1.1), J4.2 (1.2)
- net Sorties/Relais2_NO: now also J4.3 (2.1), J4.4 (2.2)
- net at D1.2 (A): now also J6.1

Commit message: avant prod
Parts:
- J4: LCSC Part # (none) -> C6391615
- J5, J6: LCSC Part # (none) -> C3816889
- U1: value SIP-4_1779205311 -> 1779205311; footprint PCM_MagIC_THT_Wurth:U_Wurth_WPME-FISM-SIP-4_1779405311 -> PCM_MagIC_THT_Wurth:U_Wurth_WPME-FISM-SIP-4_1779205311; LCSC Part # (none) -> C6652237
Connections:
- net Entrée/Input1: now also J6.4; no longer J6.3
- net Entrée/Input2: now also J6.3; no longer J6.4
- net Sorties/Output1: now also J5.3; no longer J5.1
- net Sorties/Output2: now also J5.1; no longer J5.3
Changed lines of the file:
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@@
 			)
 		)
+		(property "LCSC Part #" "C3816889"
+			(at 33.02 90.17 0)
+			(hide yes)
+			(show_name no)
+			(do_not_autoplace no)
+			(effects
+				(font
+					(size 1.27 1.27)
+				)
+			)
+		)
 		(pin "2"
 		)
@@
 			)
 		)
+		(property "LCSC Part #" "C3816889"
+			(at 33.02 33.02 0)
+			(hide yes)
+			(show_name no)
+			(do_not_autoplace no)
+			(effects
+				(font
+					(size 1.27 1.27)
+				)
+			)
+		)
 		(pin "2"
 		)
@@
 			)
 		)
+		(property "LCSC Part #" "C6391615"
+			(at 44.45 139.7 0)
+			(hide yes)
+			(show_name no)
+			(do_not_autoplace no)
+			(effects
+				(font
+					(size 1.27 1.27)
+				)
+			)
+		)
 		(pin "1"
 		)
@@
 			)
 		)
-		(property "Value" "SIP-4_1779205311"
+		(property "Value" "1779205311"
 			(at 127 49.53 0)
 			(hide yes)
@@
 			)
 		)
-		(property "Footprint" "PCM_MagIC_THT_Wurth:U_Wurth_WPME-FISM-SIP-4_1779405311"
+		(property "Footprint" "PCM_MagIC_THT_Wurth:U_Wurth_WPME-FISM-SIP-4_1779205311"
 			(at 139.7 24.13 0)
 			(hide yes)
@@
 			)
 		)
+		(property "LCSC Part #" "C6652237"
+			(at 127 44.45 0)
+			(hide yes)
+			(show_name no)
+			(do_not_autoplace no)
+			(effects
+				(font
+					(size 1.27 1.27)
+				)
+			)
+		)
 		(pin "2"
 		)
@@
 			)
 		)
-		(pin "Output1" output
+		(pin "Output2" output
 			(at 67.31 120.65 180)
 			(effects
@@
 			)
 		)
-		(pin "Output2" output
+		(pin "Output1" output
 			(at 67.31 123.19 180)
 			(effects
@@
 			)
 		)
-		(pin "Input1" input
+		(pin "Input2" input
 			(at 67.31 78.74 180)
 			(effects
@@
 			)
 		)
-		(pin "Input2" input
+		(pin "Input1" input
 			(at 67.31 83.82 180)
 			(effects
