File: puissance.kicad_sch (KiCad schematic)
At the start: 13 parts, among them J3 MEC1-110-02-F-D-A, J4 1705566, J5 1725672, J6 1725672, U1 1779205311

Commit message: MAJ post prod
Other:
- title: (none) -> Carte puissance
- moved on the sheet: D1, D2, F1
Changed lines of the file:
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@@
 	(generator_version "10.0")
 	(paper "A4")
+	(title_block
+		(title "Carte puissance")
+		(date "2026-08-17")
+		(rev "0.2")
+	)
 	(rectangle
 		(start 15.24 19.05)
-		(end 49.53 196.85)
+		(end 49.53 161.29)
 		(stroke
 			(width 0)
@@
 	)
 	(rectangle
-		(start 54.61 20.32)
+		(start 60.96 20.32)
 		(end 185.42 63.5)
 		(stroke
@@
 	)
 	(junction
-		(at 90.17 33.02)
+		(at 96.52 33.02)
 		(diameter 0)
 		(color 0 0 0 0)
@@
 	)
 	(junction
-		(at 76.2 33.02)
+		(at 80.01 33.02)
 		(diameter 0)
 		(color 0 0 0 0)
 	)
 	(junction
-		(at 142.24 52.07)
+		(at 96.52 41.91)
 		(diameter 0)
 		(color 0 0 0 0)
 	)
 	(junction
-		(at 96.52 41.91)
+		(at 142.24 52.07)
 		(diameter 0)
 		(color 0 0 0 0)
@@
 	(wire
 		(pts
-			(xy 147.32 33.02) (xy 147.32 41.91)
+			(xy 142.24 33.02) (xy 142.24 41.91)
 		)
 		(stroke
@@
 	(wire
 		(pts
-			(xy 33.02 33.02) (xy 57.15 33.02)
+			(xy 33.02 33.02) (xy 60.96 33.02)
 		)
 		(stroke
@@
 	(wire
 		(pts
-			(xy 90.17 41.91) (xy 96.52 41.91)
-		)
-		(stroke
-			(width 0)
-			(type default)
-		)
-	)
-	(wire
-		(pts
 			(xy 44.45 139.7) (xy 67.31 139.7)
 		)
@@
 	(wire
 		(pts
-			(xy 147.32 41.91) (xy 142.24 41.91)
-		)
-		(stroke
-			(width 0)
-			(type default)
-		)
-	)
-	(wire
-		(pts
 			(xy 33.02 95.25) (xy 45.72 95.25)
 		)
@@
 	(wire
 		(pts
-			(xy 90.17 41.91) (xy 90.17 33.02)
+			(xy 96.52 41.91) (xy 96.52 33.02)
 		)
 		(stroke
@@
 	(wire
 		(pts
-			(xy 72.39 33.02) (xy 76.2 33.02)
+			(xy 76.2 33.02) (xy 80.01 33.02)
 		)
 		(stroke
@@
 	(wire
 		(pts
-			(xy 76.2 33.02) (xy 90.17 33.02)
+			(xy 80.01 33.02) (xy 96.52 33.02)
 		)
 		(stroke
@@
 	(symbol
 		(lib_id "power:+24V")
-		(at 90.17 33.02 0)
+		(at 96.52 33.02 0)
 		(unit 1)
 		(body_style 1)
@@
 		(fields_autoplaced yes)
 		(property "Reference" "#PWR053"
-			(at 90.17 36.83 0)
+			(at 96.52 36.83 0)
 			(hide yes)
 			(show_name no)
@@
 		)
 		(property "Value" "+24V"
-			(at 90.17 27.94 0)
+			(at 96.52 27.94 0)
 			(show_name no)
 			(do_not_autoplace no)
@@
 		)
 		(property "Footprint" ""
-			(at 90.17 33.02 0)
+			(at 96.52 33.02 0)
 			(hide yes)
 			(show_name no)
@@
 		)
 		(property "Datasheet" ""
-			(at 90.17 33.02 0)
+			(at 96.52 33.02 0)
 			(hide yes)
 			(show_name no)
@@
 		)
 		(property "Description" "Power symbol creates a global label with name \"+24V\""
-			(at 90.17 33.02 0)
+			(at 96.52 33.02 0)
 			(hide yes)
 			(show_name no)
@@
 	(symbol
 		(lib_id "Device:D")
-		(at 60.96 33.02 180)
+		(at 64.77 33.02 180)
 		(unit 1)
 		(body_style 1)
@@
 		(fields_autoplaced yes)
 		(property "Reference" "D1"
-			(at 60.96 29.21 0)
+			(at 64.77 29.21 0)
 			(show_name no)
 			(do_not_autoplace no)
@@
 		)
 		(property "Value" "FR1G"
-			(at 60.96 29.21 0)
+			(at 64.77 29.21 0)
 			(hide yes)
 			(show_name no)
@@
 		)
 		(property "Footprint" "Diode_SMD:D_SMA"
-			(at 60.96 33.02 0)
+			(at 64.77 33.02 0)
 			(hide yes)
 			(show_name no)
@@
 		)
 		(property "Datasheet" ""
-			(at 60.96 33.02 0)
+			(at 64.77 33.02 0)
 			(hide yes)
 			(show_name no)
@@
 		)
 		(property "Description" "Diode"
-			(at 60.96 33.02 0)
+			(at 64.77 33.02 0)
 			(hide yes)
 			(show_name no)
@@
 		)
 		(property "Sim.Device" "D"
-			(at 60.96 33.02 0)
+			(at 64.77 33.02 0)
 			(hide yes)
 			(show_name no)
@@
 		)
 		(property "Sim.Pins" "1=K 2=A"
-			(at 60.96 33.02 0)
+			(at 64.77 33.02 0)
 			(hide yes)
 			(show_name no)
@@
 		)
 		(property "LCSC Part #" "C412437"
-			(at 60.96 33.02 0)
+			(at 64.77 33.02 0)
 			(hide yes)
 			(show_name no)
@@
 		)
 		(property "px_1" "0,095"
-			(at 60.96 33.02 0)
+			(at 64.77 33.02 0)
 			(hide yes)
 			(show_name no)
@@
 		)
 		(property "px_10" "0.066"
-			(at 60.96 33.02 0)
+			(at 64.77 33.02 0)
 			(hide yes)
 			(show_name no)
@@
 		)
 		(property "MPN" "FR1G"
-			(at 60.96 33.02 0)
+			(at 64.77 33.02 0)
 			(hide yes)
 			(show_name no)
@@
 	(symbol
 		(lib_id "PCM_Diode_TVS_AKL:SMAJ33CA")
-		(at 76.2 38.1 90)
+		(at 80.01 38.1 90)
 		(mirror x)
 		(unit 1)
@@
 		(dnp no)
 		(property "Reference" "D2"
-			(at 73.66 36.8299 90)
+			(at 77.47 36.8299 90)
 			(show_name no)
 			(do_not_autoplace no)
@@
 		)
 		(property "Value" "SMAJ33CA"
-			(at 73.66 39.3699 90)
+			(at 77.47 39.3699 90)
 			(show_name no)
 			(do_not_autoplace no)
@@
 		)
 		(property "Footprint" "PCM_Diode_SMD_AKL:D_SMA_TVS"
-			(at 76.2 38.1 0)
+			(at 80.01 38.1 0)
 			(hide yes)
 			(show_name no)
@@
 		)
 		(property "Datasheet" "https://www.tme.eu/Document/dbc72d81c249fe51b6ab42300e8e06d0/SMAJ_ser.pdf"
-			(at 76.2 38.1 0)
+			(at 80.01 38.1 0)
 			(hide yes)
 			(show_name no)
@@
 		)
 		(property "Description" "SMA Bidirectional TVS Diode, 33V, 400W, Alternate KiCAD Library"
-			(at 76.2 38.1 0)
+			(at 80.01 38.1 0)
 			(hide yes)
 			(show_name no)
@@
 		)
 		(property "px_1" "0,318"
-			(at 76.2 38.1 90)
+			(at 80.01 38.1 90)
 			(hide yes)
 			(show_name no)
@@
 		)
 		(property "px_10" "0.297"
-			(at 76.2 38.1 90)
+			(at 80.01 38.1 90)
 			(hide yes)
 			(show_name no)
@@
 		)
 		(property "MPN" "824501331"
-			(at 76.2 38.1 90)
+			(at 80.01 38.1 90)
 			(hide yes)
 			(show_name no)
@@
 	(symbol
 		(lib_id "Device:Fuse")
-		(at 68.58 33.02 90)
+		(at 72.39 33.02 90)
 		(unit 1)
 		(body_style 1)
@@
 		(fields_autoplaced yes)
 		(property "Reference" "F1"
-			(at 68.58 26.67 90)
+			(at 72.39 26.67 90)
 			(show_name no)
 			(do_not_autoplace no)
@@
 		)
 		(property "Value" "100mA"
-			(at 68.58 29.21 90)
+			(at 72.39 29.21 90)
 			(show_name no)
 			(do_not_autoplace no)
@@
 		)
 		(property "Footprint" "Fuse:Fuse_1210_3225Metric"
-			(at 68.58 34.798 90)
+			(at 72.39 34.798 90)
 			(hide yes)
 			(show_name no)
@@
 		)
 		(property "Datasheet" ""
-			(at 68.58 33.02 0)
+			(at 72.39 33.02 0)
 			(hide yes)
 			(show_name no)
@@
 		)
 		(property "Description" "Fuse"
-			(at 68.58 33.02 0)
+			(at 72.39 33.02 0)
 			(hide yes)
 			(show_name no)
@@
 		)
 		(property "px_1" "0,155 "
-			(at 68.58 33.02 90)
+			(at 72.39 33.02 90)
 			(hide yes)
 			(show_name no)
@@
 		)
 		(property "px_10" "0.114"
-			(at 68.58 33.02 90)
+			(at 72.39 33.02 90)
 			(hide yes)
 			(show_name no)
@@
 		)
 		(property "MPN" "0ZCH0010FF2E"
-			(at 68.58 33.02 90)
+			(at 72.39 33.02 90)
 			(hide yes)
 			(show_name no)
@@
 	(symbol
 		(lib_id "power:GND2")
-		(at 76.2 43.18 0)
+		(at 80.01 43.18 0)
 		(unit 1)
 		(body_style 1)
@@
 		(fields_autoplaced yes)
 		(property "Reference" "#PWR056"
-			(at 76.2 49.53 0)
+			(at 80.01 49.53 0)
 			(hide yes)
 			(show_name no)
@@
 		)
 		(property "Value" "GND2"
-			(at 76.2 48.26 0)
+			(at 80.01 48.26 0)
 			(show_name no)
 			(do_not_autoplace no)
@@
 		)
 		(property "Footprint" ""
-			(at 76.2 43.18 0)
+			(at 80.01 43.18 0)
 			(hide yes)
 			(show_name no)
@@
 		)
 		(property "Datasheet" ""
-			(at 76.2 43.18 0)
+			(at 80.01 43.18 0)
 			(hide yes)
 			(show_name no)
@@
 		)
 		(property "Description" "Power symbol creates a global label with name \"GND2\" , ground"
-			(at 76.2 43.18 0)
+			(at 80.01 43.18 0)
 			(hide yes)
 			(show_name no)
@@
 	(symbol
 		(lib_id "power:+5VD")
-		(at 147.32 33.02 0)
+		(at 142.24 33.02 0)
 		(unit 1)
 		(body_style 1)
@@
 		(fields_autoplaced yes)
 		(property "Reference" "#PWR054"
-			(at 147.32 36.83 0)
+			(at 142.24 36.83 0)
 			(hide yes)
 			(show_name no)
@@
 		)
 		(property "Value" "+5VD"
-			(at 147.32 27.94 0)
+			(at 142.24 27.94 0)
 			(show_name no)
 			(do_not_autoplace no)
@@
 		)
 		(property "Footprint" ""
-			(at 147.32 33.02 0)
+			(at 142.24 33.02 0)
 			(hide yes)
 			(show_name no)
@@
 		)
 		(property "Datasheet" ""
-			(at 147.32 33.02 0)
+			(at 142.24 33.02 0)
 			(hide yes)
 			(show_name no)
@@
 		)
 		(property "Description" "Power symbol creates a global label with name \"+5VD\""
-			(at 147.32 33.02 0)
+			(at 142.24 33.02 0)
 			(hide yes)
 			(show_name no)
@@
 			(project "puissance"
 				(path "/b2e6993f-467e-4b42-9c79-23dbe0260143"
-					(page "2")
+					(page "3")
 				)
 			)
@@
 			(project "puissance"
 				(path "/b2e6993f-467e-4b42-9c79-23dbe0260143"
-					(page "1")
+					(page "2")
 				)
 			)
@@
 	(sheet_instances
 		(path "/"
-			(page "10")
+			(page "1")
 		)
 	)
